File: VESC/ESC1.kicad_sch (KiCad schematic)
At the start: 36 parts, among them Q1 SP40N03GNJ, Q10 SP40N03GNJ, Q17 SP40N03GNJ, Q18 SP40N03GNJ, Q5 SP40N03GNJ, Q9 SP40N03GNJ, U4 AT32F421G8U7, U8 NSG2065Q

Commit message: Revision_2 of VESC
Parts:
- added C71: 1uF, Capacitor_SMD:C_0201_0603Metric, symbol Device:C
- C67: value 100nF -> 470uF
- R17, R29, R41: value 10K -> 75K
Connections:
- net +3.3V: now also C71.1
- net GND: now also C71.2
Other:
- moved on the sheet: FB1
Changed lines of the file:
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@@
 	)
 	(junction
+		(at 27.94 63.5)
+		(diameter 0)
+		(color 0 0 0 0)
+	)
+	(junction
 		(at 260.35 124.46)
 		(diameter 0)
@@
 	(wire
 		(pts
+			(xy 27.94 63.5) (xy 38.1 63.5)
+		)
+		(stroke
+			(width 0)
+			(type default)
+		)
+	)
+	(wire
+		(pts
 			(xy 96.52 123.19) (xy 96.52 130.81)
 		)
@@
 	(wire
 		(pts
-			(xy 35.56 63.5) (xy 38.1 63.5)
+			(xy 45.72 63.5) (xy 48.26 63.5)
 		)
 		(stroke
@@
 	)
 	(label "VDDA"
-		(at 38.1 63.5 0)
+		(at 48.26 63.5 0)
 		(effects
 			(font
@@
 			)
 		)
-		(property "Value" "10K"
+		(property "Value" "75K"
 			(at 264.16 36.8299 0)
 			(show_name no)
@@
 		(in_pos_files yes)
 		(dnp no)
-		(fields_autoplaced yes)
 		(property "Reference" "R13"
-			(at 156.21 33.02 90)
+			(at 156.21 34.036 90)
 			(show_name no)
 			(do_not_autoplace no)
@@
 		)
 		(property "Value" "220"
-			(at 156.21 35.56 90)
+			(at 156.21 36.576 90)
 			(show_name no)
 			(do_not_autoplace no)
@@
 	(symbol
 		(lib_id "power:GND")
+		(at 27.94 71.12 0)
+		(unit 1)
+		(body_style 1)
+		(exclude_from_sim no)
+		(in_bom yes)
+		(on_board yes)
+		(in_pos_files yes)
+		(dnp no)
+		(fields_autoplaced yes)
+		(property "Reference" "#PWR0105"
+			(at 27.94 77.47 0)
+			(hide yes)
+			(show_name no)
+			(do_not_autoplace no)
+			(effects
+				(font
+					(size 1.27 1.27)
+				)
+			)
+		)
+		(property "Value" "GND"
+			(at 27.94 76.2 0)
+			(show_name no)
+			(do_not_autoplace no)
+			(effects
+				(font
+					(size 1.27 1.27)
+				)
+			)
+		)
+		(property "Footprint" ""
+			(at 27.94 71.12 0)
+			(hide yes)
+			(show_name no)
+			(do_not_autoplace no)
+			(effects
+				(font
+					(size 1.27 1.27)
+				)
+			)
+		)
+		(property "Datasheet" ""
+			(at 27.94 71.12 0)
+			(hide yes)
+			(show_name no)
+			(do_not_autoplace no)
+			(effects
+				(font
+					(size 1.27 1.27)
+				)
+			)
+		)
+		(property "Description" "Power symbol creates a global label with name \"GND\" , ground"
+			(at 27.94 71.12 0)
+			(hide yes)
+			(show_name no)
+			(do_not_autoplace no)
+			(effects
+				(font
+					(size 1.27 1.27)
+				)
+			)
+		)
+		(pin "1"
+		)
+		(instances
+			(project "VENDETTAESC"
+				(path "/62497189-72eb-441b-9043-ca0a95596c6f/7c9e156b-b536-46fa-851a-311dd633243a"
+					(reference "#PWR0107")
+					(unit 1)
+				)
+				(path "/62497189-72eb-441b-9043-ca0a95596c6f/c4194d8a-4081-4750-8aa5-45e80972e9ea"
+					(reference "#PWR0105")
+					(unit 1)
+				)
+				(path "/62497189-72eb-441b-9043-ca0a95596c6f/c6d0038e-73b1-4107-979d-7d477f3b42f0"
+					(reference "#PWR0108")
+					(unit 1)
+				)
+				(path "/62497189-72eb-441b-9043-ca0a95596c6f/f855ef8c-a86d-4f49-b472-4c306de56e33"
+					(reference "#PWR0106")
+					(unit 1)
+				)
+			)
+		)
+	)
+	(symbol
+		(lib_id "power:GND")
 		(at 148.59 77.47 0)
 		(unit 1)
@@
 	)
 	(symbol
+		(lib_id "Device:C")
+		(at 27.94 67.31 0)
+		(unit 1)
+		(body_style 1)
+		(exclude_from_sim no)
+		(in_bom yes)
+		(on_board yes)
+		(in_pos_files yes)
+		(dnp no)
+		(fields_autoplaced yes)
+		(property "Reference" "C71"
+			(at 31.75 66.0399 0)
+			(show_name no)
+			(do_not_autoplace no)
+			(effects
+				(font
+					(size 1.27 1.27)
+				)
+				(justify left)
+			)
+		)
+		(property "Value" "1uF"
+			(at 31.75 68.5799 0)
+			(show_name no)
+			(do_not_autoplace no)
+			(effects
+				(font
+					(size 1.27 1.27)
+				)
+				(justify left)
+			)
+		)
+		(property "Footprint" "Capacitor_SMD:C_0201_0603Metric"
+			(at 28.9052 71.12 0)
+			(hide yes)
+			(show_name no)
+			(do_not_autoplace no)
+			(effects
+				(font
+					(size 1.27 1.27)
+				)
+			)
+		)
+		(property "Datasheet" ""
+			(at 27.94 67.31 0)
+			(hide yes)
+			(show_name no)
+			(do_not_autoplace no)
+			(effects
+				(font
+					(size 1.27 1.27)
+				)
+			)
+		)
+		(property "Description" "Unpolarized capacitor"
+			(at 27.94 67.31 0)
+			(hide yes)
+			(show_name no)
+			(do_not_autoplace no)
+			(effects
+				(font
+					(size 1.27 1.27)
+				)
+			)
+		)
+		(pin "1"
+		)
+		(pin "2"
+		)
+		(instances
+			(project "VENDETTAESC"
+				(path "/62497189-72eb-441b-9043-ca0a95596c6f/7c9e156b-b536-46fa-851a-311dd633243a"
+					(reference "C73")
+					(unit 1)
+				)
+				(path "/62497189-72eb-441b-9043-ca0a95596c6f/c4194d8a-4081-4750-8aa5-45e80972e9ea"
+					(reference "C71")
+					(unit 1)
+				)
+				(path "/62497189-72eb-441b-9043-ca0a95596c6f/c6d0038e-73b1-4107-979d-7d477f3b42f0"
+					(reference "C74")
+					(unit 1)
+				)
+				(path "/62497189-72eb-441b-9043-ca0a95596c6f/f855ef8c-a86d-4f49-b472-4c306de56e33"
+					(reference "C72")
+					(unit 1)
+				)
+			)
+		)
+	)
+	(symbol
 		(lib_id "power:GND")
 		(at 209.55 66.04 0)
@@
 			)
 		)
-		(property "Value" "100nF"
+		(property "Value" "470uF"
 			(at 26.67 132.0799 0)
 			(show_name no)
@@
 			)
 		)
-		(property "Value" "10K"
+		(property "Value" "75K"
 			(at 212.09 36.8299 0)
 			(show_name no)
@@
 	(symbol
 		(lib_id "Device:FerriteBead")
-		(at 31.75 63.5 90)
+		(at 41.91 63.5 90)
 		(unit 1)
 		(body_style 1)
@@
 		(dnp no)
 		(property "Reference" "FB1"
-			(at 32.258 68.58 90)
+			(at 42.418 68.58 90)
 			(show_name no)
 			(do_not_autoplace no)
@@
 		)
 		(property "Value" "FerriteBead"
-			(at 32.258 71.12 90)
+			(at 42.418 71.12 90)
 			(show_name no)
 			(do_not_autoplace no)
@@
 		)
 		(property "Footprint" "Inductor_SMD:L_0201_0603Metric"
-			(at 31.75 65.278 90)
+			(at 41.91 65.278 90)
 			(hide yes)
 			(show_name no)
@@
 		)
 		(property "Datasheet" ""
-			(at 31.75 63.5 0)
+			(at 41.91 63.5 0)
 			(hide yes)
 			(show_name no)
@@
 		)
 		(property "Description" "Ferrite bead"
-			(at 31.75 63.5 0)
+			(at 41.91 63.5 0)
 			(hide yes)
 			(show_name no)
@@
 			)
 		)
-		(property "Value" "10K"
+		(property "Value" "75K"
 			(at 238.76 36.8299 0)
 			(show_name no)
