File: VESC/ESC1.kicad_sch (KiCad schematic)
At the start: 44 parts, among them Q1 SP40N03GNJ, Q10 SP40N03GNJ, Q17 SP40N03GNJ, Q18 SP40N03GNJ, Q5 SP40N03GNJ, Q9 SP40N03GNJ, U4 AT32F421G8U7, U8 NSG2065Q

Commit message: Rev 2.0 fabrication documentation
Parts:
- C11, C15, C19, C23, C59, C63, C75: Distributor Link (none) -> https://www.lcsc.com/product-detail/C77020.html?spm=wm.fly.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; LCSC (none) -> C77020; MANUFACTURER (none) -> muRata; Manufacturer Part Number (none) -> GRM155R71H104KE14D
- C67: Distributor Link (none) -> https://www.lcsc.com/product-detail/C19666.html?spm=wm.fly.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; LCSC (none) -> C19666; MANUFACTURER (none) -> Samsung Electro-Mechanics; Manufacturer Part Number (none) -> CL10A475KO8NNNC
- C71: Distributor Link (none) -> https://www.lcsc.com/product-detail/C29266.html?spm=wm.fly.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; LCSC (none) -> C29266; MANUFACTURER (none) -> Samsung Electro-Mechanics; Manufacturer Part Number (none) -> CL05A105KO5NNNC
- C87, C88, C89: Distributor Link (none) -> https://www.lcsc.com/product-detail/C7209937.html?spm=wm.fl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; LCSC (none) -> C7209937; MANUFACTURER (none) -> YAGEO; Manufacturer Part Number (none) -> AC0402KRX7R0BB221
- FB1: Distributor Link (none) -> https://www.lcsc.com/product-detail/C124089.html?s_z=n_q_t_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; LCSC (none) -> C124089; MANUFACTURER (none) -> FH; Manufacturer Part Number (none) -> CBW100505U101T
- Q1, Q10, Q17, Q18, Q5, Q9: Distributor Link (none) -> https://www.lcsc.com/product-detail/C22466709.html?s_z=n_q_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; LCSC (none) -> C22466709; MANUFACTURER (none) -> Siliup; Manufacturer Part Number (none) -> SP40N03GNJ
- R13: Distributor Link (none) -> https://www.lcsc.com/product-detail/C25152.html?spm=wm.fly.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; LCSC (none) -> C25152; MANUFACTURER (none) -> UNI-ROYAL; Manufacturer Part Number (none) -> 0402WGJ0220TCE
- R17, R25, R29, R31, R41, R43, R9: Distributor Link (none) -> https://www.lcsc.com/product-detail/C60489.html?spm=wm.fly.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; LCSC (none) -> C60489; MANUFACTURER (none) -> YAGEO; Manufacturer Part Number (none) -> RC0402JR-0710KL
- R21, R30, R42, R5: Distributor Link (none) -> https://www.lcsc.com/product-detail/C106235.html?spm=wm.fly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; LCSC (none) -> C106235; MANUFACTURER (none) -> YAGEO; Manufacturer Part Number (none) -> RC0402FR-071KL
- R53, R57, R61, R62, R69, R70: Distributor Link (none) -> https://www.lcsc.com/product-detail/C25083.html?spm=wm.fly.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; LCSC (none) -> C25083; MANUFACTURER (none) -> UNI-ROYAL; Manufacturer Part Number (none) -> 0402WGF150JTCE
- R90, R91, R92: Distributor Link (none) -> https://www.lcsc.com/product-detail/C25169.html?spm=wm.fly.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; LCSC (none) -> C25169; MANUFACTURER (none) -> UNI-ROYAL; Manufacturer Part Number (none) -> 0402WGJ047JTCE
- TP3, TP7: Distributor Link (none) -> -; LCSC (none) -> -; MANUFACTURER (none) -> -; Manufacturer Part Number (none) -> -
- U4: Distributor Link (none) -> https://www.lcsc.com/product-detail/C2765098.html?s_z=s_p_A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; LCSC (none) -> C2765098; MANUFACTURER (none) -> ARTERY; Manufacturer Part Number (none) -> AT32F421G8U7
- U8: Distributor Link (none) -> https://www.lcsc.com/product-detail/C41414478.html?s_z=n_q_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; MANUFACTURER (none) -> WXNSIC; Manufacturer Part Number (none) -> NSG2065Q
