File: VESC/VENDETTAESC.kicad_pcb (KiCad board)
At the start: 6 copper layers, 40.5 x 43 mm, 203 parts, among them J6 SM08B-SRSS-TB, Q1 SP40N03GNJ, Q10 SP40N03GNJ, Q11 SP40N03GNJ, Q12 SP40N03GNJ, Q13 SP40N03GNJ, Q14 SP40N03GNJ, Q15 SP40N03GNJ, Q16 SP40N03GNJ, Q17 SP40N03GNJ, Q18 SP40N03GNJ, Q19 SP40N03GNJ, Q2 SP40N03GNJ, Q20 SP40N03GNJ, Q21 SP40N03GNJ, Q22 SP40N03GNJ, Q23 SP40N03GNJ, Q24 SP40N03GNJ, Q3 SP40N03GNJ, Q4 SP40N03GNJ, Q5 SP40N03GNJ, Q6 SP40N03GNJ, Q7 SP40N03GNJ, Q8 SP40N03GNJ, Q9 SP40N03GNJ, U1 INA185, U10 NSG2065Q, U11 NSG2065Q, U12 VESC, U2 LMR51420YDDCR, U3 TLV76733DRVx, U4 AT32F421G8U7, U5 AT32F421G8U7, U6 AT32F421G8U7, U7 AT32F421G8U7, U8 NSG2065Q, U9 NSG2065Q

Commit message: Revision_2 of VESC
Parts:
- added D1: SMBJ30A, SMBJ30A:DIOM4336X265N, F.Cu at (199.8, 117.0)
- moved C5 5.85 mm to (194.2, 117.0)
- moved C4 5.80 mm to (192.6, 117.0)
- moved U3 4.95 mm to (190.3, 117.1)
- moved R3 2.95 mm to (198.7, 117.8)
- moved R1 1.87 mm to (199.7, 110.0)
- moved G*** 1.63 mm to (187.4, 116.9)
- moved G*** 1.46 mm to (212.0, 117.0)
- moved R4 0.53 mm to (200.8, 117.8)
- moved C69 0.51 mm to (212.6, 94.3)
- moved Q15 0.46 mm to (209.8, 105.2)
- moved G*** 0.32 mm to (195.3, 117.1)
- moved C6 0.27 mm to (203.9, 114.6)
- moved G*** 0.20 mm to (204.3, 117.2)
- moved L1 0.19 mm to (203.9, 113.6)
- moved C10 0.10 mm to (194.1, 114.6)
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Routing:
- net +8V: track 99.8 -> 0.06 mm, vias 4 -> 38
- net +BATT: track 158.7 -> 60.5 mm, vias 28 -> 36
- net GND: track 181.1 -> 159.1 mm, vias 140 -> 274
- net Net-(Q17-G): track 5.62 -> 19.7 mm, vias 1 -> 2
- net Net-(Q21-G): track 28.5 -> 15.6 mm, vias 1 -> 2
- net /ESC3/MOTORA: track 12.1 -> 24.5 mm, vias 2 -> 3
- net /ESC4/MOTORC: track 4.04 -> 13.2 mm, vias 0 -> 2
- net /ESC3/MOTORB: track 29.7 -> 21.4 mm, vias 1 -> 4
- net /ESC4/MOTORA: track 34.6 -> 26.6 mm, vias 1 -> 3
- net Net-(Q10-G): track 18.3 -> 10.6 mm, vias 1 -> 2
- net /ESC1/MOTORC: track 7.61 -> 14.4 mm, vias 0 -> 3
- net /ESC2/MOTORB: track 19.2 -> 13.4 mm, vias 1 -> 2
- net Net-(Q19-G): track 20.4 -> 14.7 mm, vias 1 -> 2
- net Net-(Q14-G): track 9.29 -> 3.59 mm
- net Net-(Q16-G): track 6.99 -> 1.33 mm
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- added copper zone on B.Cu, net +3.3V
- added copper zone on In3.Cu, net +8V
- added copper zone on In2.Cu, net GND
- added copper zone on B.Cu, net Net-(U2-CB)
- added copper zone on B.Cu, net Net-(U2-FB)
- added copper zone on B.Cu, net Net-(U2-SW)
- removed copper zone on In2.Cu, net +BATT

Commit message: Revision_2 of VESC
Parts:
- added C71: 1uF, Capacitor_SMD:C_0201_0603Metric, B.Cu at (198.0, 96.9)
- added C72: 1uF, Capacitor_SMD:C_0201_0603Metric, B.Cu at (198.2, 108.9)
- added C73: 1uF, Capacitor_SMD:C_0201_0603Metric, B.Cu at (201.3, 95.7)
- added C74: 1uF, Capacitor_SMD:C_0201_0603Metric, B.Cu at (201.1, 107.0)
- C67, C68, C69, C70: value 100nF -> 470uF
- R1: value 0.2mR -> 0.5mR
- R17, R18, R19, R20, R29, R32, R35, R38, R41, R44, R47, R50: value 10K -> 75K
- R3: value 124K -> 95k3
- turned D1 to 180 degrees
Connections:
- D1 pad A: GND -> /CSA+
- D1 pad C: /CSA+ -> GND
Routing:
- net +3.3V: track 103.2 -> 106.4 mm
- net GND: track 159.1 -> 161.0 mm, vias 274 -> 294
