File: VESC/VENDETTAESC.kicad_pcb (KiCad board)
At the start: 6 copper layers, 40.5 x 43 mm, 236 parts, among them J6 SM08B-SRSS-TB, Q1 SP40N03GNJ, Q10 SP40N03GNJ, Q11 SP40N03GNJ, Q12 SP40N03GNJ, Q13 SP40N03GNJ, Q14 SP40N03GNJ, Q15 SP40N03GNJ, Q16 SP40N03GNJ, Q17 SP40N03GNJ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

Commit message: VFC Revision 2.0
Parts:
- moved C63 0.07 mm to (185.6, 90.9)
- moved R29 0.07 mm to (195.3, 100.1)
- moved Q23 0.07 mm to (209.9, 109.8)
Routing:
- net +3.3V: track 119.7 -> 121.0 mm, vias 29 -> 31
- net /ESC2/MOTORC: track 17.4 -> 18.4 mm
- net GND: track 136.1 -> 135.5 mm, vias 377 -> 383
