File: VESC/VENDETTAESC.kicad_sch (KiCad schematic)
At the start: 52 parts, among them J6 SM08B-SRSS-TB, U1 INA185, U12 VESC, U2 LMR51420YDDCR, U3 TLV76733DRVx

Commit message: Revision_2 of VESC
Parts:
- added D1: SMBJ30A, SMBJ30A:DIOM4336X265N, symbol SMBJ30A:SMBJ30A
Connections:
- net CSA+: now also D1.C
- net GND: now also D1.A

Commit message: Revision_2 of VESC
Parts:
- R1: value 0.2mR -> 0.5mR
- R3: value 124K -> 95k3
Connections:
- net CSA+: now also D1.A; no longer D1.C
- net GND: now also D1.C; no longer D1.A
Other:
- moved on the sheet: D1
Changed lines of the file:
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@@
 			)
 		)
-		(property "Value" "124K"
+		(property "Value" "95k3"
 			(at 252.73 45.7199 0)
 			(show_name no)
@@
 	(symbol
 		(lib_id "SMBJ30A:SMBJ30A")
-		(at 106.68 73.66 0)
+		(at 106.68 73.66 180)
 		(unit 1)
 		(body_style 1)
@@
 			)
 		)
-		(property "Value" "0.2mR"
+		(property "Value" "0.5mR"
 			(at 92.71 74.93 90)
 			(show_name no)

Commit message: Revision_1 of VFC complete
Other:
- note added: "Edge Connectors"
Changed lines of the file:
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@@
 	(generator_version "10.0")
 	(paper "A4")
+	(text ""
+		(exclude_from_sim no)
+		(at 34.798 20.32 0)
+		(effects
+			(font
+				(size 2.54 2.54)
+			)
+		)
+	)
+	(text ""
+		(exclude_from_sim no)
+		(at 28.194 20.828 0)
+		(effects
+			(font
+				(size 2.54 2.54)
+			)
+		)
+	)
+	(text "Edge Connectors"
+		(exclude_from_sim no)
+		(at 42.672 21.336 0)
+		(effects
+			(font
+				(size 2.54 2.54)
+			)
+		)
+	)
 	(junction
 		(at 104.14 139.7)
@@
 		)
 	)
+	(polyline
+		(pts
+			(xy 182.88 76.2) (xy 182.88 121.92)
+		)
+		(stroke
+			(width 0)
+			(type default)
+		)
+	)
 	(wire
 		(pts
@@
 		)
 	)
+	(polyline
+		(pts
+			(xy 279.4 121.92) (xy 279.4 76.2)
+		)
+		(stroke
+			(width 0)
+			(type default)
+		)
+	)
 	(wire
 		(pts
@@
 	(polyline
 		(pts
+			(xy 182.88 121.92) (xy 279.4 121.92)
+		)
+		(stroke
+			(width 0)
+			(type default)
+		)
+	)
+	(polyline
+		(pts
 			(xy 182.88 22.86) (xy 182.88 25.4)
 		)
@@
 		)
 		(stroke
+			(width 0)
+			(type default)
+		)
+	)
+	(polyline
+		(pts
+			(xy 182.88 76.2) (xy 279.4 76.2)
+		)
+		(stroke
