File: VESC/VENDETTAESC.kicad_sch (KiCad schematic)
At the start: 53 parts, among them J6 SM08B-SRSS-TB, U1 INA185, U12 VESC, U2 LMR51420YDDCR, U3 TLV76733DRVx

Commit message: Added fabrication files
Parts:
- L1: value 1mH -> 4.7uH; footprint Inductor_SMD:L_0402_1005Metric -> Inductor_SMD:L_0603_1608Metric; LCSC (none) -> C46594347
- R3: value 95k3 -> 124K
Connections:
- net +8V renamed +10V
Changed lines of the file:
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@@
 	)
 	(junction
-		(at 201.93 95.25)
-		(diameter 0)
-		(color 0 0 0 0)
-	)
-	(junction
 		(at 78.74 158.75)
 		(diameter 0)
@@
 	)
 	(junction
+		(at 201.93 95.25)
+		(diameter 0)
+		(color 0 0 0 0)
+	)
+	(junction
 		(at 271.78 40.64)
 		(diameter 0)
@@
 			)
 		)
-		(property "Value" "1mH"
+		(property "Value" "4.7uH"
 			(at 243.84 38.1 90)
 			(show_name no)
@@
 			)
 		)
-		(property "Footprint" "Inductor_SMD:L_0402_1005Metric"
+		(property "Footprint" "Inductor_SMD:L_0603_1608Metric"
 			(at 243.84 40.64 0)
 			(hide yes)
@@
 			)
 		)
+		(property "LCSC" "C46594347"
+			(at 243.84 40.64 90)
+			(hide yes)
+			(show_name no)
+			(do_not_autoplace no)
+			(effects
+				(font
+					(size 1.27 1.27)
+				)
+			)
+		)
 		(pin "2"
 		)
@@
 			)
 		)
-		(property "Value" "95k3"
+		(property "Value" "124K"
 			(at 252.73 45.7199 0)
 			(show_name no)
@@
 		(in_pos_files yes)
 		(dnp no)
-		(fields_autoplaced yes)
 		(property "Reference" "#PWR014"
 			(at 271.78 44.45 0)
@@
 			)
 		)
-		(property "Value" "+8V"
-			(at 271.78 35.56 0)
+		(property "Value" "+10V"
+			(at 269.24 35.814 0)
 			(show_name no)
 			(do_not_autoplace no)
@@
 					(size 1.27 1.27)
 				)
+				(justify left)
 			)
 		)
@@
 	)
 	(symbol
+		(lib_id "power:+8V")
+		(at 201.93 95.25 0)
+		(unit 1)
+		(body_style 1)
+		(exclude_from_sim no)
+		(in_bom yes)
+		(on_board yes)
+		(in_pos_files yes)
+		(dnp no)
+		(property "Reference" "#PWR015"
+			(at 201.93 99.06 0)
+			(hide yes)
+			(show_name no)
+			(do_not_autoplace no)
+			(effects
+				(font
+					(size 1.27 1.27)
+				)
+			)
+		)
+		(property "Value" "+10V"
+			(at 198.374 90.17 0)
+			(show_name no)
+			(do_not_autoplace no)
+			(effects
+				(font
+					(size 1.27 1.27)
+				)
+				(justify left)
+			)
+		)
+		(property "Footprint" ""
+			(at 201.93 95.25 0)
+			(hide yes)
+			(show_name no)
+			(do_not_autoplace no)
+			(effects
+				(font
+					(size 1.27 1.27)
+				)
+			)
+		)
+		(property "Datasheet" ""
+			(at 201.93 95.25 0)
+			(hide yes)
+			(show_name no)
+			(do_not_autoplace no)
+			(effects
+				(font
+					(size 1.27 1.27)
+				)
+			)
+		)
+		(property "Description" "Power symbol creates a global label with name \"+8V\""
+			(at 201.93 95.25 0)
+			(hide yes)
+			(show_name no)
+			(do_not_autoplace no)
+			(effects
+				(font
+					(size 1.27 1.27)
+				)
+			)
+		)
+		(pin "1"
+		)
+		(instances
+			(project "VENDETTAESC"
+				(path "/62497189-72eb-441b-9043-ca0a95596c6f"
+					(reference "#PWR015")
+					(unit 1)
+				)
+			)
+		)
+	)
+	(symbol
 		(lib_id "Device:R")
 		(at 250.19 54.61 180)
@@
 					(unit 1)
 				)
-			)
-		)
-	)
-	(symbol
-		(lib_id "power:+8V")
-		(at 201.93 95.25 0)
-		(unit 1)
-		(body_style 1)
-		(exclude_from_sim no)
-		(in_bom yes)
-		(on_board yes)
-		(in_pos_files yes)
-		(dnp no)
-		(fields_autoplaced yes)
-		(property "Reference" "#PWR015"
-			(at 201.93 99.06 0)
-			(hide yes)
-			(show_name no)
-			(do_not_autoplace no)
-			(effects
-				(font
-					(size 1.27 1.27)
-				)
-			)
-		)
-		(property "Value" "+8V"
-			(at 201.93 90.17 0)
-			(show_name no)
-			(do_not_autoplace no)
-			(effects
-				(font
-					(size 1.27 1.27)
-				)
-			)
-		)
-		(property "Footprint" ""
-			(at 201.93 95.25 0)
-			(hide yes)
-			(show_name no)
-			(do_not_autoplace no)
-			(effects
-				(font
-					(size 1.27 1.27)
-				)
-			)
-		)
-		(property "Datasheet" ""
-			(at 201.93 95.25 0)
-			(hide yes)
-			(show_name no)
-			(do_not_autoplace no)
-			(effects
-				(font
-					(size 1.27 1.27)
-				)
-			)
-		)
-		(property "Description" "Power symbol creates a global label with name \"+8V\""
-			(at 201.93 95.25 0)
-			(hide yes)
-			(show_name no)
-			(do_not_autoplace no)
-			(effects
-				(font
-					(size 1.27 1.27)
-				)
-			)
-		)
-		(pin "1"
-		)
-		(instances
-			(project "VENDETTAESC"
-				(path "/62497189-72eb-441b-9043-ca0a95596c6f"
-					(reference "#PWR015")
-					(unit 1)
-				)

Commit message: Routing improvements
Parts:
- removed L1: 4.7uH, Inductor_SMD:L_0603_1608Metric, symbol Device:L
- added L1: 10uH, Inductor_SMD:L_Changjiang_FTC404020S, symbol FAUL0530-100MT:FXL0530-100-M
Connections:
- net +10V: now also L1.1
- net at C6.1, U2.2 (SW): now also L1.2
- net TEL: now reaches J6.4
- net TEL: now also U12.19 (TX)
- no-connect marks 2 -> 0
Other:
- moved on the sheet: C6, U2

Commit message: Added telemetery feature for ESC
Parts:
- added R77: 10K, Resistor_SMD:R_0201_0603Metric, symbol Device:R
Connections:
- net +3.3V: now also R77.2
- net TEL: now also R77.1
Changed lines of the file:
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@@
 	(wire
 		(pts
+			(xy 124.46 24.13) (xy 128.27 24.13)
+		)
+		(stroke
+			(width 0)
+			(type default)
+		)
+	)
+	(wire
+		(pts
 			(xy 48.26 92.71) (xy 48.26 95.25)
 		)
@@
 	(wire
 		(pts
+			(xy 143.51 22.86) (xy 143.51 24.13)
+		)
+		(stroke
+			(width 0)
+			(type default)
+		)
+	)
+	(wire
+		(pts
 			(xy 101.6 73.66) (xy 99.06 73.66)
 		)
@@
 	(wire
 		(pts
+			(xy 143.51 24.13) (xy 135.89 24.13)
+		)
+		(stroke
+			(width 0)
+			(type default)
+		)
+	)
+	(wire
+		(pts
 			(xy 104.14 124.46) (xy 118.11 124.46)
 		)
@@
 		)
 	)
+	(global_label "TEL"
+		(shape input)
+		(at 124.46 24.13 180)
+		(fields_autoplaced yes)
+		(effects
+			(font
+				(size 1.27 1.27)
+			)
+			(justify right)
+		)
+		(property "Intersheetrefs" "${INTERSHEET_REFS}"
+			(at 118.3301 24.13 0)
+			(hide yes)
+			(show_name no)
+			(do_not_autoplace no)
+			(effects
+				(font
+					(size 1.27 1.27)
+				)
+				(justify right)
+			)
+		)
+	)
 	(global_label "CURR"
 		(shape input)
@@
 	)
 	(symbol
+		(lib_id "power:+3.3V")
+		(at 143.51 22.86 0)
+		(unit 1)
+		(body_style 1)
+		(exclude_from_sim no)
+		(in_bom yes)
+		(on_board yes)
+		(in_pos_files yes)
+		(dnp no)
+		(fields_autoplaced yes)
+		(property "Reference" "#PWR0109"
+			(at 143.51 26.67 0)
+			(hide yes)
+			(show_name no)
+			(do_not_autoplace no)
+			(effects
+				(font
+					(size 1.27 1.27)
+				)
+			)
+		)
+		(property "Value" "+3.3V"
+			(at 143.51 17.78 0)
+			(show_name no)
+			(do_not_autoplace no)
+			(effects
+				(font
+					(size 1.27 1.27)
+				)
+			)
+		)
+		(property "Footprint" ""
+			(at 143.51 22.86 0)
+			(hide yes)
+			(show_name no)
+			(do_not_autoplace no)
+			(effects
+				(font
+					(size 1.27 1.27)
+				)
+			)
+		)
+		(property "Datasheet" ""
+			(at 143.51 22.86 0)
+			(hide yes)
+			(show_name no)
+			(do_not_autoplace no)
+			(effects
+				(font
+					(size 1.27 1.27)
+				)
+			)
+		)
+		(property "Description" "Power symbol creates a global label with name \"+3.3V\""
+			(at 143.51 22.86 0)
+			(hide yes)
+			(show_name no)
+			(do_not_autoplace no)
+			(effects
+				(font
+					(size 1.27 1.27)
+				)
+			)
+		)
+		(pin "1"
+		)
+		(instances
+			(project "VENDETTAESC"
+				(path "/62497189-72eb-441b-9043-ca0a95596c6f"
+					(reference "#PWR0109")
+					(unit 1)
+				)
+			)
+		)
+	)
+	(symbol
 		(lib_id "Device:C")
 		(at 118.11 128.27 0)
@@
 					(unit 1)
 				)
+			)
+		)
+	)
+	(symbol
+		(lib_id "Device:R")
+		(at 132.08 24.13 90)
+		(unit 1)
+		(body_style 1)
+		(exclude_from_sim no)
+		(in_bom yes)
+		(on_board yes)
+		(in_pos_files yes)
+		(dnp no)
+		(fields_autoplaced yes)
+		(property "Reference" "R77"
+			(at 132.08 17.78 90)
+			(show_name no)
+			(do_not_autoplace no)
+			(effects
+				(font
+					(size 1.27 1.27)
+				)
+			)
+		)
+		(property "Value" "10K"
+			(at 132.08 20.32 90)
+			(show_name no)
+			(do_not_autoplace no)
+			(effects
+				(font
+					(size 1.27 1.27)
+				)
+			)
+		)
+		(property "Footprint" "Resistor_SMD:R_0201_0603Metric"
+			(at 132.08 25.908 90)
+			(hide yes)
+			(show_name no)
+			(do_not_autoplace no)
+			(effects
+				(font
+					(size 1.27 1.27)
+				)
+			)
+		)
+		(property "Datasheet" ""
+			(at 132.08 24.13 0)
+			(hide yes)
+			(show_name no)
+			(do_not_autoplace no)
+			(effects
+				(font
+					(size 1.27 1.27)
+				)
+			)
+		)
+		(property "Description" "Resistor"
+			(at 132.08 24.13 0)
+			(hide yes)
+			(show_name no)
+			(do_not_autoplace no)
+			(effects
+				(font
+					(size 1.27 1.27)
+				)
+			)
+		)
+		(pin "1"
+		)
+		(pin "2"
+		)
+		(instances
+			(project "VENDETTAESC"
+				(path "/62497189-72eb-441b-9043-ca0a95596c6f"
+					(reference "R77")
+					(unit 1)
+				)

Commit message: VESC Revision 2.0
Parts:
- C1, C2, C3, C6, C7, C8: footprint Capacitor_SMD:C_0201_0603Metric -> Capacitor_SMD:C_0402_1005Metric
- C10: footprint Capacitor_SMD:C_0402_1005Metric -> Capacitor_SMD:C_0805_2012Metric
- C4, C5: footprint Capacitor_SMD:C_0603_1608Metric -> Capacitor_SMD:C_0805_2012Metric
- C9: value 22uF -> 4.7uF; footprint Capacitor_SMD:C_0402_1005Metric -> Capacitor_SMD:C_0603_1608Metric
- R2, R3, R4, R77: footprint Resistor_SMD:R_0201_0603Metric -> Resistor_SMD:R_0402_1005Metric
Changed lines of the file:
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@@
 			)
 		)
-		(property "Footprint" "Capacitor_SMD:C_0402_1005Metric"
+		(property "Footprint" "Capacitor_SMD:C_0805_2012Metric"
 			(at 267.6652 102.87 0)
 			(hide yes)
@@
 			)
 		)
-		(property "Value" "22uF"
+		(property "Value" "4.7uF"
 			(at 259.08 100.3299 0)
 			(show_name no)
@@
 			)
 		)
-		(property "Footprint" "Capacitor_SMD:C_0402_1005Metric"
+		(property "Footprint" "Capacitor_SMD:C_0603_1608Metric"
 			(at 256.2352 102.87 0)
 			(hide yes)
@@
 			)
 		)
-		(property "Footprint" "Capacitor_SMD:C_0603_1608Metric"
+		(property "Footprint" "Capacitor_SMD:C_0805_2012Metric"
 			(at 261.3152 52.07 0)
 			(hide yes)
@@
 			)
 		)
-		(property "Footprint" "Resistor_SMD:R_0201_0603Metric"
+		(property "Footprint" "Resistor_SMD:R_0402_1005Metric"
 			(at 251.968 44.45 90)
 			(hide yes)
@@
 			)
 		)
-		(property "Footprint" "Capacitor_SMD:C_0201_0603Metric"
+		(property "Footprint" "Capacitor_SMD:C_0402_1005Metric"
 			(at 242.2652 102.87 0)
 			(hide yes)
@@
 			)
 		)
-		(property "Footprint" "Capacitor_SMD:C_0201_0603Metric"
+		(property "Footprint" "Capacitor_SMD:C_0402_1005Metric"
 			(at 26.3652 90.17 0)
 			(hide yes)
@@
 			)
 		)
-		(property "Footprint" "Capacitor_SMD:C_0201_0603Metric"
+		(property "Footprint" "Capacitor_SMD:C_0402_1005Metric"
 			(at 202.8952 102.87 0)
 			(hide yes)
@@
 			)
 		)
-		(property "Footprint" "Capacitor_SMD:C_0201_0603Metric"
+		(property "Footprint" "Capacitor_SMD:C_0402_1005Metric"
 			(at 54.3052 104.14 0)
 			(hide yes)
@@
 			)
 		)
-		(property "Footprint" "Capacitor_SMD:C_0201_0603Metric"
+		(property "Footprint" "Capacitor_SMD:C_0402_1005Metric"
 			(at 187.6552 46.99 0)
 			(hide yes)
@@
 			)
 		)
-		(property "Footprint" "Capacitor_SMD:C_0201_0603Metric"
+		(property "Footprint" "Capacitor_SMD:C_0402_1005Metric"
 			(at 222.25 35.2552 0)
 			(hide yes)
@@
 			)
 		)
-		(property "Footprint" "Resistor_SMD:R_0201_0603Metric"
+		(property "Footprint" "Resistor_SMD:R_0402_1005Metric"
 			(at 35.56 79.502 90)
 			(hide yes)
@@
 			)
 		)
-		(property "Footprint" "Resistor_SMD:R_0201_0603Metric"
+		(property "Footprint" "Resistor_SMD:R_0402_1005Metric"
 			(at 132.08 25.908 90)
 			(hide yes)
@@
 			)
 		)
-		(property "Footprint" "Capacitor_SMD:C_0603_1608Metric"
+		(property "Footprint" "Capacitor_SMD:C_0805_2012Metric"
 			(at 272.7452 52.07 0)
 			(hide yes)
@@
 			)
 		)
-		(property "Footprint" "Resistor_SMD:R_0201_0603Metric"
+		(property "Footprint" "Resistor_SMD:R_0402_1005Metric"
 			(at 251.968 54.61 90)
 			(hide yes)

Commit message: Rev 2.0 fabrication documentation
Parts:
- C1, C2, C3, C6, C7, C8: Distributor Link (none) -> https://www.lcsc.com/product-detail/C77020.html?spm=wm.fly.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; LCSC (none) -> C77020; MANUFACTURER (none) -> muRata; Manufacturer Part Number (none) -> GRM155R71H104KE14D
- C10, C4, C5: Distributor Link (none) -> https://www.lcsc.com/product-detail/C602037.html?spm=wm.fly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; LCSC (none) -> C602037; MANUFACTURER (none) -> Samsung Electro-Mechanics; Manufacturer Part Number (none) -> CL21A226MAYNNNE
- C27, C28, C29, C30, C31, C32, C33, C34, C35, C36, C37, C38, C39, C40, C41, C42, C43, C44, C45, C46, C47, C48, C49, C50, C51, C52, C53, C54, C55, C56, C57, C58: Distributor Link (none) -> https://www.lcsc.com/product-detail/C2932476.html?s_z=n_q_C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; LCSC (none) -> C2932476; MANUFACTURER (none) -> Samsung Electro-Mechanics; Manufacturer Part Number (none) -> CL21A106KBYQNNE
- C9: Distributor Link (none) -> https://www.lcsc.com/product-detail/C19666.html?spm=wm.fly.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; LCSC (none) -> C19666; MANUFACTURER (none) -> Samsung Electro-Mechanics; Manufacturer Part Number (none) -> CL10A475KO8NNNC
- D1: Distributor Link (none) -> https://www.lcsc.com/product-detail/C135065.html?s_z=s_p_SM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; LCSC (none) -> C135065; MANUFACTURER Taiwan Semiconductor -> DIODES; Manufacturer Part Number (none) -> SMBJ30A-13-F
- J6: Distributor Link (none) -> https://www.lcsc.com/product-detail/C160407.html?s_z=n_q_C1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; LCSC (none) -> C160407; Manufacturer Part Number (none) -> SM08B-SRSS-TB(LF)(SN)
- L1: Distributor Link (none) -> https://www.lcsc.com/product-detail/C53198553.html?s_z=s_p_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; LCSC (none) -> C53198553; MANUFACTURER (none) -> FAUKU; Manufacturer Part Number (none) -> GXTC0420-100-MT
- R1: Distributor Link (none) -> https://www.lcsc.com/product-detail/C19679480.html?spm=wm.f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; LCSC (none) -> C19679480; MANUFACTURER (none) -> RESI; Manufacturer Part Number (none) -> EBWM2512JL500S9
- R2: Distributor Link (none) -> https://www.lcsc.com/product-detail/C106235.html?spm=wm.fly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; LCSC (none) -> C106235; MANUFACTURER (none) -> YAGEO; Manufacturer Part Number (none) -> RC0402FR-071KL
- R3: Distributor Link (none) -> https://www.lcsc.com/product-detail/C36777.html?spm=wm.fly.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; LCSC (none) -> C36777; MANUFACTURER (none) -> UNI-ROYAL; Manufacturer Part Number (none) -> 0402WGF1243TCE
- R4, R77: Distributor Link (none) -> https://www.lcsc.com/product-detail/C60489.html?spm=wm.fly.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; LCSC (none) -> C60489; MANUFACTURER (none) -> YAGEO; Manufacturer Part Number (none) -> RC0402JR-0710KL
- U1: value INA185 -> INA185A2; Distributor Link (none) -> https://www.lcsc.com/product-detail/C2059320.html?s_z=s_p_I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; LCSC (none) -> C2059320; MANUFACTURER (none) -> Texas Instruments; Manufacturer Part Number (none) -> INA185A2IDRLR
- U12: Distributor Link (none) -> -; LCSC (none) -> -; MANUFACTURER (none) -> -; Manufacturer Part Number (none) -> -
- U2: value LMR51420YDDCR -> LMR51420YFDDCR; Distributor Link (none) -> https://www.lcsc.com/product-detail/C7296200.html?s_z=n_q_C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; LCSC (none) -> C7296200; Manufacturer Part Number (none) -> LMR51420YFDDCR
- U3: Distributor Link (none) -> https://www.lcsc.com/product-detail/C2848334.html?s_z=n_q_C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; LCSC (none) -> C2848334; MANUFACTURER (none) -> Texas Instruments; Manufacturer Part Number (none) -> TLV76733DRVR
