File: VFC/VENDETTAFC.kicad_pcb (KiCad board)
At the start: 6 copper layers, 40.5 x 43 mm, 161 parts, among them J1 SM06B-SRSS-TB_LF__SN_, J10 SM04B-SRSS-TB_LF__SN_, J11 SM04B-SRSS-TB_LF__SN_, J12 SM03B-SRSS-TB_LF__SN_, J2 USB4940-00-A_REVA, J3 SM03B-SRSS-TB_LF__SN_, J5 SM03B-SRSS-TB_LF__SN_, J6 SM08B-SRSS-TB_LF__SN_, J7 SM03B-SRSS-TB_LF__SN_, J8 SM03B-SRSS-TB_LF__SN_, J9 SM06B-SRSS-TB_LF__SN_, Q2 AO3400A, U1 STM32F722RETx, U10 USBLC6-2SC6, U2 BMP388, U3 AP2112K-3.3TRG1, U5 ESP32-C3, U6 ICM-42688-P, U7 W25N04KVZEIR, Y2 C3E-40.000-10-1015-X-R, Y3 C3E-8.000-18-3030-X-R

Commit message: VFC PCB traces update
Parts:
- removed the REF** at (185.5, 54.5)
- removed the REF** at (155.0, 85.0)
- removed the REF** at (185.5, 85.0)
- added ?: , , F.Cu at (185.5, 54.5)
- added ?: , , F.Cu at (155.0, 85.0)
- added ?: , , F.Cu at (185.5, 85.0)
- added C24: 1uF, Capacitor_SMD:C_0402_1005Metric, B.Cu at (171.6, 82.6)
- added C25: 1uF, Capacitor_SMD:C_0402_1005Metric, B.Cu at (171.4, 79.9)
- added FL2: 220 Ohms @ 100 MHz, BLM18PG221SN1D:BEADC1608X95N, B.Cu at (171.9, 78.7)
- added U11: AP7361C-FGE-7, AP7361C-FGE-7:SON65P300X300X63-9N, B.Cu at (179.2, 59.1)
- C12, C13: value 1uF -> 4.7uF
- FL1: value 120 -> 120Ω @ 100MHz
- U3: value AP2112K-3.3TRG1 -> NCP167BMX330TBG; footprint AP2112K-3.3TRG1:SOT95P285X140-5N -> NCP167BMX330TBG:VREG_NCP167BMX330TBG
- moved U3 22.5 mm to (171.5, 81.3), turned to -90 degrees
- moved R29 5.15 mm to (158.1, 60.7), turned to 90 degrees
- moved C12 4.72 mm to (180.1, 56.5), turned to 0 degrees
- moved TP18 3.40 mm to (177.8, 87.0)
- moved R25 3.34 mm to (174.1, 80.2), turned to 180 degrees
- moved C13 3.28 mm to (179.3, 61.7), turned to 180 degrees
- moved D7 3.24 mm to (164.5, 77.5)
- moved TP17 3.20 mm to (174.6, 87.0)
- moved C15 2.45 mm to (167.6, 82.7)
- moved C19 2.45 mm to (163.2, 78.2)
- moved C22 2.45 mm to (163.7, 81.5)
- moved D8 2.45 mm to (160.2, 81.5)
- moved R14 2.45 mm to (166.0, 83.2)
- moved R15 2.45 mm to (165.0, 83.2)
- moved C21 2.45 mm to (161.7, 78.2)
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Connections:
- C10 pad 1: +3.3V -> +3.3VA
- C11 pad 1: +3.3V -> +3.3VA
- C28 pad 1: +3.3V -> +3.3VA
- C4 pad 1: +3.3V -> +3.3VA
- C6 pad 1: +3.3V -> +3.3VA
- C7 pad 1: +3.3V -> +3.3VA
- C9 pad 1: +3.3V -> +3.3VA
- FL1 pad 2: +3.3V -> +3.3VA
- R12 pad 2: +3.3V -> +3.3VA
- R25 pad 2: +3.3V -> +3.3VA
- R26 pad 2: +3.3V -> +3.3VA
- R4 pad 1: +3.3V -> +3.3VA
- U1 pad 10: unconnected-(U1-PC2-Pad10) -> LED3
- U1 pad 16: M4 -> M1
- U1 pad 17: M3 -> M2
- U1 pad 2: ADC_CUR -> U_LED
- U1 pad 20: LED3 -> ADC_CUR
- U1 pad 25: M2 -> M3
- U1 pad 26: M1 -> M4
- U1 pad 29: U_LED -> unconnected-(U1-PB11-Pad29)
- U2 pad 1: +3.3V -> +3.3VA
- U2 pad 10: +3.3V -> +3.3VA
- U2 pad 6: +3.3V -> +3.3VA
- U3 pad 1: +5V -> Net-(U3-OUT)
- U3 pad 4: (no net) -> +5V
- U3 pad 5: +3.3V -> GND
- U6 pad 5: +3.3V -> +3.3VA
- U6 pad 8: +3.3V -> +3.3VA
Routing:
- net +3.3V: track 0.00 -> 43.3 mm, vias 0 -> 31
- net GND: track 0.00 -> 41.0 mm, vias 0 -> 91
- net UART7_RX: track 0.00 -> 36.5 mm, vias 0 -> 3
- net UART7_TX: track 0.00 -> 36.3 mm, vias 0 -> 3
- net /BOOT0: track 0.00 -> 36.2 mm, vias 0 -> 2
- net GPS_SDA: track 0.00 -> 35.0 mm, vias 0 -> 3
- net +3.3VA: track 0.00 -> 33.9 mm, vias 0 -> 9
- net GPS_SCL: track 0.00 -> 30.5 mm, vias 0 -> 3
- net LED1: track 0.00 -> 28.6 mm, vias 0 -> 4
- net UART4_RX: track 0.00 -> 27.3 mm, vias 0 -> 2
- net UART6_RX: track 0.00 -> 26.5 mm, vias 0 -> 2
- net LED2: track 0.00 -> 26.2 mm, vias 0 -> 5
- net UART6_TX: track 0.00 -> 25.9 mm, vias 0 -> 2
- net UART5_TX: track 0.00 -> 24.6 mm, vias 0 -> 3
- net UART5_RX: track 0.00 -> 24.5 mm, vias 0 -> 3
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- added copper zone on B.Cu, net +3.3V
- added copper zone on F.Cu, net +3.3V
- added copper zone on In3.Cu, net +3.3V
- added copper zone on B.Cu, net +3.3VA
- added copper zone on F.Cu, net +3.3VA
- added copper zone on B.Cu, net +5V
- added copper zone on In3.Cu, net +5V
- added copper zone on B.Cu, net +5VBAT
- added copper zone on F.Cu, net +5VBUS
- added copper zone on B.Cu, net +9V
- added copper zone on B.Cu, net +VLIPO
- added copper zone on In3.Cu, net +VLIPO
- added copper zone on B.Cu, net ADC_CUR
- added copper zone on B.Cu, net ESC_RX
- added copper zone on B.Cu, net GND
- added copper zone on F.Cu, net GND
- added copper zone on In1.Cu, net GND
- added copper zone on In2.Cu, net GND
- added copper zone on In3.Cu, net GND
- added copper zone on In4.Cu, net GND
- added copper zone on B.Cu, net M1
- added copper zone on B.Cu, net M2
- added copper zone on B.Cu, net M3
- added copper zone on B.Cu, net M4
- added copper zone on F.Cu, net Net-(C32-Pad1)
- added copper zone on B.Cu, net Net-(U3-OUT)
- added copper zone on B.Cu, net Net-(U4-SW)
- added copper zone on B.Cu, net Net-(U9-SW)

Commit message: Revision_1 of VFC complete
Parts:
- added G***: LOGO, silkscreen.preety:arrow, F.Cu at (163.9, 66.0)
- added G***: LOGO, drawings:KNIFE_F, B.Cu at (159.8, 54.8)
- added G***: LOGO, drawings:VLOGO, B.Cu at (162.2, 61.9)
- added G***: LOGO, drawings:KNIFE_F, B.Cu at (180.4, 54.5)
- moved U8 10.3 mm to (191.9, 61.0), turned to 90 degrees
- moved TP2 2.43 mm to (182.6, 65.9)
- moved Y2 1.26 mm to (182.8, 68.5)
- moved Y3 0.66 mm to (182.8, 72.4)
- moved C33 0.31 mm to (187.9, 66.1)
- moved C34 0.31 mm to (187.0, 66.1)
- moved TP1 0.25 mm to (180.8, 65.8)
- moved J6 0.16 mm to (170.3, 53.3)
Routing:
- net UART4_TX: track 0.00 -> 17.6 mm, vias 0 -> 3
- net GND: track 41.0 -> 53.0 mm, vias 91 -> 93
- net +5VBUS: track 0.00 -> 4.61 mm, vias 7 -> 9
- net Net-(U5-GPIO21/U0TXD): track 4.63 -> 1.93 mm
- net +5V: track 15.0 -> 17.6 mm, vias 15 -> 24
- net Net-(R7-Pad1): track 0.00 -> 2.47 mm
- net /HSE_OUT: track 6.28 -> 4.41 mm
- net /HSE_IN: track 6.26 -> 4.49 mm
- net /Sensor Section/CLK_OUT: track 3.93 -> 5.41 mm
- net LED4: track 18.0 -> 19.2 mm
- net /Sensor Section/CLK_IN: track 4.66 -> 5.50 mm
- net /Sensor Section/ANT: track 4.18 -> 3.63 mm
- net +3.3V: vias 31 -> 29
- added copper zone on F.Cu, net +5V
- added copper zone on In1.Cu, net +5V
- added copper zone on In2.Cu, net +5V
- added copper zone on In4.Cu, net +5V
- added copper zone on B.Cu, net +5VBUS
- added copper zone on In2.Cu, net +5VBUS
- added copper zone on In3.Cu, net +5VBUS
Other:
- board size 40.5 x 43 mm -> 43.5 x 43 mm
- board text added: "+5V"
- board text added: "+5V GND"
- board text added: "+5V GND U7_RX"
- board text added: "+9V"
- board text added: "+9V GND U3_TX"
- board text added: "-BUZZ"
- board text added: "BOOT"
- board text added: "BUZZER"
- board text added: "DJI"
- board text added: "G"
- board text added: "GND"
- board text added: "GND -BUZZ"
- board text added: "GPS"
- board text added: "G_SCL"
- board text added: "G_SDA"
- board text added: "L1"
- board text added: "L2"
- board text added: "L3"
- board text added: "L4"
- board text added: "LED1"
- board text added: "LED2"
- board text added: "LED3"
- board text added: "LED4"
- board text added: "LEDs"
- board text added: "M4 M3 M2 M1"
- board text added: "M4 M3 M2 M1 RX CUR GND VESC"
- board text added: "RECEIVER"
- board text added: "TX CUR GND VESC"
- board text added: "U3_RX"
- board text added: "U3_RX GND U4_RX"
- board text added: "U3_TX"
- board text added: "U4_RX"
- board text added: "U4_TX"
- board text added: "U5_RX"
- board text added: "U5_TX"
- board text added: "U5_TX U5_RX"
- board text added: "U6_RX"
- board text added: "U6_RX U6_TX"
- board text added: "U6_TX"
- board text added: "U7_RX"
- board text added: "U7_TX"
- board text added: "U7_TX G_SDA G_SCL"
- board text added: "UART5"
- board text added: "VENDETTA FC F7"
