File: VFC/VENDETTAFC.kicad_pcb (KiCad board)
At the start: 6 copper layers, 43.5 x 43 mm, 169 parts, among them J1 SM06B-SRSS-TB_LF__SN_, J10 SM04B-SRSS-TB_LF__SN_, J11 SM04B-SRSS-TB_LF__SN_, J12 SM03B-SRSS-TB_LF__SN_, J2 USB4940-00-A_REVA, J3 SM03B-SRSS-TB_LF__SN_, J5 SM03B-SRSS-TB_LF__SN_, J6 SM08B-SRSS-TB_LF__SN_, J7 SM03B-SRSS-TB_LF__SN_, J8 SM03B-SRSS-TB_LF__SN_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

Commit message: LICENSE
Parts:
- removed R19, R30: 10K, Resistor_SMD:R_0402_1005Metric
- added R6: 10K, Resistor_SMD:R_0402_1005Metric, F.Cu at (188.4, 59.7)
- moved TP1 5.17 mm to (178.8, 61.1)
- moved TP2 4.72 mm to (178.8, 63.1)
Connections:
- TP1 pad 1: Net-(U5-GPIO20/U0RXD) -> Net-(U5-GPIO13/SPIWP)
- TP2 pad 1: Net-(U5-GPIO21/U0TXD) -> Net-(U5-GPIO14/SPICS0)
- U1 pad 11: ESP_CS -> ESP_BOOT
- U1 pad 21: ESP_SCK -> ESP_EN
- U1 pad 22: ESP_MISO -> ESP_TX
- U1 pad 23: ESP_MOSI -> ESP_RX
- U5 pad 15: Net-(U5-GPIO9) -> ESP_BOOT
- U5 pad 20: ESP_CS -> Net-(U5-GPIO13/SPIWP)
- U5 pad 21: ESP_MISO -> Net-(U5-GPIO14/SPICS0)
- U5 pad 22: ESP_SCK -> unconnected-(U5-GPIO15/SPICLK-Pad22)
- U5 pad 23: ESP_MOSI -> unconnected-(U5-GPIO16/SPID-Pad23)
- U5 pad 27: Net-(U5-GPIO20/U0RXD) -> ESP_TX
- U5 pad 28: Net-(U5-GPIO21/U0TXD) -> ESP_RX
- U5 pad 7: +3.3V -> ESP_EN
Routing:
- net ESP_EN: track 0.00 -> 19.0 mm, vias 0 -> 2
- net ESP_RX: track 0.00 -> 11.4 mm
- net ESP_TX: track 0.00 -> 11.3 mm
- net ESP_BOOT: track 0.00 -> 10.9 mm, vias 0 -> 2
- net ESP_CS: track 10.2 -> 0.00 mm, vias 2 -> 0
- net ESP_MISO: track 9.44 -> 0.00 mm
- net ESP_SCK: track 8.71 -> 0.00 mm
- net ESP_MOSI: track 8.54 -> 0.00 mm
- net Net-(U5-GPIO14/SPICS0): track 0.00 -> 3.27 mm
- net Net-(U5-GPIO20/U0RXD): track 3.15 -> 0.00 mm
- net Net-(U5-GPIO13/SPIWP): track 0.00 -> 3.04 mm
- net Net-(U5-GPIO21/U0TXD): track 1.93 -> 0.00 mm
- net +3.3V: track 43.3 -> 44.6 mm
- net Net-(U5-GPIO9): track 1.17 -> 0.00 mm
- net ADC_CUR: track 7.30 -> 6.59 mm
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
Commit message: Added fabrication files
Parts:
- moved FL1 0.66 mm to (176.1, 66.1), turned to 0 degrees
Routing:
- net M1: track 13.4 -> 16.1 mm
- net ESP_EN: track 19.0 -> 20.9 mm
- net UART4_TX: track 17.6 -> 19.1 mm
- net Net-(U1-VDDA): track 1.56 -> 2.85 mm
- net ESP_BOOT: track 10.9 -> 11.9 mm
- net LED3: track 21.9 -> 22.7 mm
- net IMU_CS: track 3.96 -> 4.61 mm
- net IMU_SCK: track 1.86 -> 2.49 mm, vias 2 -> 1
- net UART5_TX: track 24.2 -> 24.7 mm
- net IMU_INT: track 6.48 -> 7.00 mm, vias 2 -> 1
- net UART5_RX: track 23.6 -> 24.1 mm
- net UART4_RX: track 27.3 -> 27.8 mm
- net GND: vias 92 -> 91
- added copper zone on In2.Cu, net +3.3V

Commit message: Routing improvements
Parts:
- removed C30, C31: 1pF, Capacitor_SMD:C_0402_1005Metric
- removed U8: ~, crossair-ca-c03-antenna-1.snapshot.1:CA-C03
- added AT1: 2450AT43B100E, 2450AT43B100E:ANTENNA_2450AT43B100E, F.Cu at (192.0, 61.0)
- L3: value 2nH -> 1.8nH
- moved L3 1.06 mm to (187.9, 64.1), turned to 90 degrees
Connections:
- J10 pad S1: GND -> unconnected-(J10-SHIELD-PadS1)_1
- J10 pad S2: GND -> unconnected-(J10-SHIELD-PadS1)
- J7 pad S1: GND -> unconnected-(J7-SHIELD-PadS1)
- J7 pad S2: GND -> unconnected-(J7-SHIELD-PadS1)_1
- U1 pad 16: M1 -> ESP_TX
- U1 pad 17: M2 -> ESP_RX
- U1 pad 21: ESP_EN -> unconnected-(U1-PA5-Pad21)
- U1 pad 22: ESP_TX -> M1
- U1 pad 23: ESP_RX -> M2
- U1 pad 8: unconnected-(U1-PC0-Pad8) -> ESP_EN
Routing:
- net GND: track 53.0 -> 37.5 mm, vias 91 -> 100
- net M1: track 16.1 -> 8.60 mm
- net ESP_TX: track 11.3 -> 5.59 mm, vias 0 -> 2
- net ESP_RX: track 11.3 -> 8.24 mm
- net M2: track 11.6 -> 8.92 mm
- net Net-(U5-LNA_IN): track 2.64 -> 1.26 mm
- net ESP_EN: track 20.9 -> 22.2 mm
Other:
- board size 43.5 x 43 mm -> 43.6 x 43 mm
