File: VFC/VENDETTAFC.kicad_pcb (KiCad board)
At the start: 6 copper layers, 43.6 x 43 mm, 166 parts, among them J1 SM06B-SRSS-TB_LF__SN_, J10 SM04B-SRSS-TB_LF__SN_, J11 SM04B-SRSS-TB_LF__SN_, J12 SM03B-SRSS-TB_LF__SN_, J2 USB4940-00-A_REVA, J3 SM03B-SRSS-TB_LF__SN_, J5 SM03B-SRSS-TB_LF__SN_, J6 SM08B-SRSS-TB_LF__SN_, J7 SM03B-SRSS-TB_LF__SN_, J8 SM03B-SRSS-TB_LF__SN_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

Commit message: Routing improvements
Parts:
- removed the G*** at (162.2, 61.9)
- removed J11: SM04B-SRSS-TB_LF__SN_, SM04B-SRSS-TB_LF__SN_:JST_SM04B-SRSS-TB_LF__SN_
- removed TP33, TP34: TestPoint, TestPoint:TestPoint_Pad_1.0x1.0mm
- added C26: 100nF, Capacitor_SMD:C_0402_1005Metric, B.Cu at (166.3, 70.3)
- added C27: 100nF, Capacitor_SMD:C_0402_1005Metric, B.Cu at (160.4, 60.4)
- added C30: 100nF, Capacitor_SMD:C_0402_1005Metric, B.Cu at (163.9, 60.4)
- added C31: 22uF, Capacitor_Tantalum_SMD:CP_EIA-1608-08_AVX-J, B.Cu at (168.2, 62.5)
- added C43: 22uF, Capacitor_Tantalum_SMD:CP_EIA-1608-08_AVX-J, B.Cu at (166.6, 60.0)
- added C44: 100nF, Capacitor_SMD:C_0402_1005Metric, B.Cu at (162.5, 60.3)
- added IC1: AT7456E, AT7456E_KiCad:SOP65P640X120-29N, B.Cu at (162.2, 65.2)
- added J13: SM04B-SRSS-TB_LF__SN_, SM04B-SRSS-TB_LF__SN_:JST_SM04B-SRSS-TB_LF__SN_, B.Cu at (163.9, 58.1)
- added J14: SM04B-SRSS-TB_LF__SN_, SM04B-SRSS-TB_LF__SN_:JST_SM04B-SRSS-TB_LF__SN_, B.Cu at (162.3, 87.5)
- added R30: 75, Resistor_SMD:R_0402_1005Metric, B.Cu at (169.5, 61.9)
- added R38: 75, Resistor_SMD:R_0402_1005Metric, B.Cu at (161.6, 60.4)
- added TP27: TestPoint, TestPoint:TestPoint_Pad_1.0x1.0mm, F.Cu at (164.4, 90.8)
- added TP28: TestPoint, TestPoint:TestPoint_Pad_1.0x1.0mm, F.Cu at (162.2, 90.8)
- added Y1: ABM8-27.000MHZ-B2-T, ABM8-27.000MHZ-B2-T:XTAL_ABM8-27.000MHZ-B2-T, B.Cu at (160.0, 71.1)
- D5: value SMBJ30A -> SMAJ5.0A; footprint SMBJ30A:DIOM4336X265N -> SMAJ5.0A:DIOM4325X250N
- L1, L2: footprint Inductor_SMD:L_0402_1005Metric -> Inductor_SMD:L_Changjiang_FTC404020S
- moved R9 5.38 mm to (182.7, 84.6)
- moved D5 4.97 mm to (162.9, 74.4), turned to 0 degrees
- moved R8 4.65 mm to (180.3, 84.6)
- moved R7 3.59 mm to (181.7, 84.6)
- moved C20 3.47 mm to (177.9, 84.5)
- moved R15 3.10 mm to (167.9, 84.4)
- moved C22 3.07 mm to (162.9, 84.5)
- moved J6 2.95 mm to (173.2, 53.3)
- moved R16 2.57 mm to (165.5, 84.5)
- moved C23 2.27 mm to (167.6, 74.0), turned to 180 degrees
- moved C40 2.06 mm to (174.6, 84.5), turned to 180 degrees
- moved D8 1.76 mm to (158.5, 81.5)
- moved C25 1.55 mm to (172.6, 79.0)
- moved C24 1.55 mm to (172.7, 81.7)
- moved FL2 1.55 mm to (173.1, 77.7)
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Connections:
- net FLS_SCK renamed FLS/OSD_SCK
- J1 pad 1: UART4_RX -> UART4_TX
- J6 pad 5: ESC_RX -> UART4_RX
- TP13 pad 1: UART4_RX -> UART4_TX
- TP9 pad 1: ESC_RX -> UART4_RX
- U1 pad 24: ESC_RX -> unconnected-(U1-PC4-Pad24)
- U1 pad 27: unconnected-(U1-PB2-Pad27) -> OSD_CS
- U1 pad 29: unconnected-(U1-PB11-Pad29) -> VIDEO_CC
- U1 pad 35: FLS_MISO -> FLS/OSD_MISO
- U1 pad 36: FLS_MOSI -> FLS/OSD_MOSI
- U1 pad 51: UART4_TX -> UART4_RX
- U1 pad 52: UART4_RX -> UART4_TX
- U7 pad 2: FLS_MISO -> FLS/OSD_MOSI
- U7 pad 5: FLS_MOSI -> FLS/OSD_MISO
Routing:
- net VIDEO_OUT: track 0.00 -> 35.2 mm, vias 0 -> 4
- net +5V: track 17.6 -> 47.1 mm, vias 24 -> 30
- net UART6_RX: track 26.5 -> 0.00 mm, vias 2 -> 0
- net UART6_TX: track 25.9 -> 0.00 mm, vias 2 -> 0
- net UART4_TX: track 19.1 -> 43.1 mm
- net FLS/OSD_MOSI: track 0.00 -> 17.7 mm, vias 0 -> 2
- net FLS/OSD_MISO: track 0.00 -> 13.3 mm, vias 0 -> 3
- net OSD_CS: track 0.00 -> 12.4 mm, vias 0 -> 2
- net FLS_MISO: track 11.5 -> 0.00 mm
- net FLS/OSD_SCK: track 7.28 -> 16.2 mm, vias 0 -> 3
- net VIDEO_CC: track 0.00 -> 8.71 mm, vias 0 -> 1
- net FLS_MOSI: track 6.49 -> 0.00 mm, vias 2 -> 0
- net LED1: track 28.7 -> 35.1 mm, vias 4 -> 2
- net M4: track 9.03 -> 15.3 mm
- net ESC_RX: track 6.20 -> 0.00 mm, vias 3 -> 0
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- added copper zone on F.Cu, net +VLIPO
- added copper zone on B.Cu, net /SG
- removed copper zone on In2.Cu, net +3.3V
- removed copper zone on B.Cu, net ADC_CUR
- removed copper zone on B.Cu, net ESC_RX
- removed copper zone on B.Cu, net M1
- removed copper zone on B.Cu, net M2
- removed copper zone on B.Cu, net M3
- removed copper zone on B.Cu, net M4

Commit message: VFC Revision 2.0
Parts:
- added C45: 0.1uF, Capacitor_SMD:C_0402_1005Metric, B.Cu at (174.7, 78.1)
- added C46: 0.1uF, Capacitor_SMD:C_0402_1005Metric, B.Cu at (159.4, 76.9)
- added C47: 0.1uF, Capacitor_SMD:C_0402_1005Metric, B.Cu at (173.6, 83.2)
- added C48: 0.1uF, Capacitor_SMD:C_0402_1005Metric, B.Cu at (160.2, 85.2)
- added C49: 100nF, Capacitor_SMD:C_0402_1005Metric, B.Cu at (174.2, 76.5)
- added C50: 100nF, Capacitor_SMD:C_0402_1005Metric, B.Cu at (179.8, 63.1)
- C12, C13: footprint Capacitor_SMD:C_0402_1005Metric -> Capacitor_SMD:C_0603_1608Metric
- C17, C19, C20, C22: footprint Capacitor_SMD:C_0603_1608Metric -> Capacitor_SMD:C_0805_2012Metric
- C18, C21: value 100uF -> 10uF; footprint Capacitor_SMD:C_0603_1608Metric -> Capacitor_SMD:C_0805_2012Metric
- C40: value 100uF -> 22uF; footprint Capacitor_SMD:C_0603_1608Metric -> Capacitor_SMD:C_0805_2012Metric
- moved R36 2.87 mm to (180.1, 75.7), turned to 0 degrees
- moved C17 1.05 mm to (178.2, 77.4)
- moved C21 0.72 mm to (160.9, 77.7)
- moved C18 0.55 mm to (176.2, 77.4)
- moved C22 0.53 mm to (162.8, 85.0)
- moved C40 0.42 mm to (174.2, 84.7)
- moved C12 0.35 mm to (181.5, 56.2)
- moved FL2 0.33 mm to (172.8, 77.8)
- moved L2 0.31 mm to (162.9, 81.7)
- moved C13 0.25 mm to (180.4, 61.9)
- moved C20 0.25 mm to (177.7, 84.7)
- moved C19 0.22 mm to (162.9, 77.7)
- moved TP1 0.15 mm to (178.7, 61.0)
- moved TP2 0.15 mm to (178.7, 63.1)
Routing:
- net GND: track 31.8 -> 26.3 mm, vias 115 -> 152
- net +VLIPO: track 2.82 -> 7.37 mm, vias 21 -> 22
- net UART7_TX: track 37.4 -> 41.5 mm
- net GPS_SDA: track 34.9 -> 38.9 mm
- net Net-(U4-EN/SYNC): track 9.64 -> 6.90 mm
- net +9V: track 14.9 -> 17.3 mm
- net +5VBAT: track 4.17 -> 6.45 mm
- net LED2: track 27.2 -> 28.2 mm
- net +5V: track 47.1 -> 47.8 mm
- net M1: track 11.8 -> 12.5 mm
- net UART4_RX: track 23.5 -> 24.1 mm
- net ADC_CUR: track 9.71 -> 10.4 mm
- net M2: track 12.5 -> 13.2 mm
- net M3: track 13.7 -> 14.3 mm
- net M4: track 15.3 -> 15.9 mm
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- added copper zone on In2.Cu, net +3.3VA
Other:
- board text added: "VENDETTA FC F7 v2.0"
- board text removed: "VENDETTA FC F7"

Commit message: VFC Revision 2.0
Routing:
- net +5V: track 47.8 -> 49.0 mm
- net UART4_TX: track 43.5 -> 44.2 mm
- net +3.3V: track 45.6 -> 46.3 mm
- net FLS_CS: track 16.4 -> 17.0 mm
