File: VFC/interface.kicad_sch (KiCad schematic)
At the start: 53 parts, among them J1 SM06B-SRSS-TB_LF__SN_, J10 SM04B-SRSS-TB_LF__SN_, J11 SM04B-SRSS-TB_LF__SN_, J12 SM03B-SRSS-TB_LF__SN_, J3 SM03B-SRSS-TB_LF__SN_, J5 SM03B-SRSS-TB_LF__SN_, J6 SM08B-SRSS-TB_LF__SN_, J7 SM03B-SRSS-TB_LF__SN_, J8 SM03B-SRSS-TB_LF__SN_, J9 SM06B-SRSS-TB_LF__SN_

Commit message: Routing improvements
Connections:
- net GND: no longer J10.S1 (SHIELD), J10.S2 (SHIELD), J7.S1 (SHIELD), J7.S2 (SHIELD)
- new net: J10.S1 (SHIELD), J10.S2 (SHIELD)
- new net: J7.S1 (SHIELD), J7.S2 (SHIELD)
- no-connect marks 2 -> 4
Changed lines of the file:
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@@
-	)
-	(junction
-		(at 223.52 226.06)
-		(diameter 0)
-		(color 0 0 0 0)
 	)
 	(junction
@@
 	)
 	(junction
-		(at 115.57 135.89)
-		(diameter 0)
-		(color 0 0 0 0)
-	)
-	(junction
 		(at 101.6 96.52)
 		(diameter 0)
@@
 	)
 	(no_connect
+		(at 218.44 226.06)
+	)
+	(no_connect
 		(at 325.12 95.25)
 	)
@@
 		(at 325.12 99.06)
 	)
+	(no_connect
+		(at 120.65 135.89)
+	)
 	(polyline
 		(pts
@@
 	(wire
 		(pts
-			(xy 115.57 135.89) (xy 115.57 139.7)
-		)
-		(stroke
-			(width 0)
-			(type default)
-		)
-	)
-	(wire
-		(pts
 			(xy 153.67 99.06) (xy 157.48 99.06)
 		)
@@
 		)
 	)
-	(wire
-		(pts
-			(xy 223.52 220.98) (xy 223.52 226.06)
-		)
-		(stroke
-			(width 0)
-			(type default)
-		)
-	)
 	(polyline
 		(pts
@@
 	(wire
 		(pts
-			(xy 218.44 226.06) (xy 223.52 226.06)
-		)
-		(stroke
-			(width 0)
-			(type default)
-		)
-	)
-	(wire
-		(pts
 			(xy 105.41 66.04) (xy 120.65 66.04)
 		)
@@
 	(wire
 		(pts
-			(xy 120.65 135.89) (xy 115.57 135.89)
-		)
-		(stroke
-			(width 0)
-			(type default)
-		)
-	)
-	(wire
-		(pts
 			(xy 311.15 95.25) (xy 325.12 95.25)
 		)
@@
 	(wire
 		(pts
-			(xy 223.52 226.06) (xy 223.52 229.87)
+			(xy 223.52 220.98) (xy 223.52 229.87)
 		)
 		(stroke
@@
 	(wire
 		(pts
-			(xy 115.57 130.81) (xy 115.57 135.89)
-		)
-		(stroke
+			(xy 115.57 130.81) (xy 115.57 139.7)
+		)
+		(stroke

Commit message: Routing improvements
Parts:
- removed J11: SM04B-SRSS-TB_LF__SN_, SM04B-SRSS-TB_LF__SN_:JST_SM04B-SRSS-TB_LF__SN_, symbol SM04B-SRSS-TB_LF__SN_:SM04B-SRSS-TB_LF__SN_
- removed TP33, TP34, TP36: TestPoint, TestPoint:TestPoint_Pad_1.0x1.0mm, symbol Connector:TestPoint
- removed TP35: TestPoint, TestPoint:TestPoint_Pad_2.0x2.0mm, symbol Connector:TestPoint
- added J13, J14: SM04B-SRSS-TB_LF__SN_, SM04B-SRSS-TB_LF__SN_:JST_SM04B-SRSS-TB_LF__SN_, symbol SM04B-SRSS-TB_LF__SN_:SM04B-SRSS-TB_LF__SN_
- added TP27, TP28: TestPoint, TestPoint:TestPoint_Pad_1.0x1.0mm, symbol Connector:TestPoint
Connections:
- net ESC_RX is gone; now on net UART4_RX: J6.5, TP9.1
- net +5V: now also J13.1, J14.4
- net GND: now also J13.2, J14.3
- net UART4_RX: no longer J1.1, TP13.1
- net UART4_TX: now also J1.1, TP13.1, J14.2, TP27.1
- new net: J14.S1 (SHIELD), J14.S2 (SHIELD)
- new net: J13.S1 (SHIELD), J13.S2 (SHIELD)
- new net VIDEO_CC: J13.4
- new net VIDEO_IN: J13.3
- new net VIDEO_OUT: J14.1, TP28.1
- no-connect marks 4 -> 6
Other:
- note added: "ANALOG VTX"
- note added: "CAM"
- note removed: "External UART"
- moved on the sheet: J12, TP37, TP38, TP39

Commit message: VFC Revision 2.0
Parts:
- C40: value 100uF -> 22uF; footprint Capacitor_SMD:C_0603_1608Metric -> Capacitor_SMD:C_0805_2012Metric
Changed lines of the file:
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@@
 			)
 		)
-		(property "Value" "100uF"
+		(property "Value" "22uF"
 			(at 105.41 101.5999 0)
 			(show_name no)
@@
 			)
 		)
-		(property "Footprint" "Capacitor_SMD:C_0603_1608Metric"
+		(property "Footprint" "Capacitor_SMD:C_0805_2012Metric"
 			(at 102.5652 104.14 0)
 			(hide yes)

Commit message: VFC Revision 2.0
Connections:
- net GND: now also J7.S1 (SHIELD), J7.S2 (SHIELD)
- no-connect marks 6 -> 5
Changed lines of the file:
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@@
+	)
+	(junction
+		(at 223.52 226.06)
+		(diameter 0)
+		(color 0 0 0 0)
 	)
 	(junction
@@
 	)
 	(no_connect
-		(at 218.44 226.06)
-	)
-	(no_connect
 		(at 265.43 160.02)
 	)
@@
 		)
 	)
+	(wire
+		(pts
+			(xy 223.52 226.06) (xy 223.52 229.87)
+		)
+		(stroke
+			(width 0)
+			(type default)
+		)
+	)
 	(polyline
 		(pts
@@
 	(wire
 		(pts
-			(xy 223.52 220.98) (xy 223.52 229.87)
+			(xy 223.52 220.98) (xy 223.52 226.06)
 		)
 		(stroke
@@
 		)
 		(stroke
+			(width 0)
+			(type default)
+		)
+	)
+	(wire
+		(pts
+			(xy 218.44 226.06) (xy 223.52 226.06)
+		)
+		(stroke

Commit message: Rev 2.0 fabrication documentation
Parts:
- added TP33, TP34, TP35, TP36: TestPoint, TestPoint:TestPoint_Pad_1.0x1.0mm, symbol Connector:TestPoint
- C40: Distributor Link (none) -> https://www.lcsc.com/product-detail/C22367832.html?spm=wm.f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; LCSC (none) -> C22367832; MANUFACTURER (none) -> Chinocera; MANUFACTURER PART NUMBER (none) -> HGC0805R5226M350NSLJ
- J1, J9: Distributor Link (none) -> https://www.lcsc.com/product-detail/C2845365.html?s_z=n_q_S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; LCSC (none) -> C2845365; MANUFACTURER JST -> HCTL; MANUFACTURER PART NUMBER (none) -> HC-1.0-6PWT
- J10, J13, J14: Distributor Link (none) -> https://www.lcsc.com/product-detail/C2845363.html?s_z=n_q_S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; LCSC (none) -> C2845363; MANUFACTURER JST -> HCTL; MANUFACTURER PART NUMBER (none) -> HC-1.0-4PWT
- J12, J3, J5, J7, J8: Distributor Link (none) -> https://www.lcsc.com/product-detail/C2845362.html?s_z=n_q_S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; LCSC (none) -> C2845362; MANUFACTURER JST -> HCTL; MANUFACTURER PART NUMBER (none) -> HC-1.0-3PWT
- J6: Distributor Link (none) -> https://www.lcsc.com/product-detail/C160407.html?s_z=n_q_SM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; LCSC (none) -> C160407; MANUFACTURER PART NUMBER (none) -> SM08B-SRSS-TB(LF)(SN)
- TP10, TP11, TP12, TP13, TP14, TP15, TP16, TP17, TP18, TP19, TP23, TP24, TP25, TP26, TP27, TP28, TP29, TP30, TP31, TP32, TP37, TP38, TP39, TP40, TP41, TP42, TP43, TP44, TP45, TP46, TP47, TP48, TP49, TP5, TP50, TP51, TP6, TP7, TP8, TP9: Distributor Link (none) -> -; LCSC (none) -> -; MANUFACTURER (none) -> -; MANUFACTURER PART NUMBER (none) -> -
Connections:
- net +VLIPO: now also TP36.1
- net VIDEO_CC: now also TP35.1
- net VIDEO_IN: now also TP34.1
- new net +3.3V: TP33.1
