File: VFC/pwr.kicad_sch (KiCad schematic)
At the start: 48 parts, among them J2 USB4940-00-A_REVA, U10 USBLC6-2SC6, U11 AP7361C-FGE-7, U3 NCP167BMX330TBG

Commit message: Routing improvements
Parts:
- removed D5: SMBJ30A, SMBJ30A:DIOM4336X265N, symbol SMBJ30A:SMBJ30A
- added D5: SMAJ5.0A, SMAJ5.0A:DIOM4325X250N, symbol SMAJ5.0A:SMAJ5.0A
- L1, L2: footprint Inductor_SMD:L_0402_1005Metric -> Inductor_SMD:L_Changjiang_FTC404020S
Connections:
- net +5VBUS: now also D5.C
- net GND: now also D5.A
Changed lines of the file:
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@@
 	)
 	(symbol
+		(lib_id "SMAJ5.0A:SMAJ5.0A")
+		(at 179.07 67.31 270)
+		(unit 1)
+		(body_style 1)
+		(exclude_from_sim no)
+		(in_bom yes)
+		(on_board yes)
+		(in_pos_files yes)
+		(dnp no)
+		(fields_autoplaced yes)
+		(property "Reference" "D5"
+			(at 181.61 66.0399 90)
+			(show_name no)
+			(do_not_autoplace no)
+			(effects
+				(font
+					(size 1.27 1.27)
+				)
+				(justify left)
+			)
+		)
+		(property "Value" "SMAJ5.0A"
+			(at 181.61 68.5799 90)
+			(show_name no)
+			(do_not_autoplace no)
+			(effects
+				(font
+					(size 1.27 1.27)
+				)
+				(justify left)
+			)
+		)
+		(property "Footprint" "SMAJ5.0A:DIOM4325X250N"
+			(at 179.07 67.31 0)
+			(hide yes)
+			(show_name no)
+			(do_not_autoplace no)
+			(effects
+				(font
+					(size 1.27 1.27)
+				)
+				(justify bottom)
+			)
+		)
+		(property "Datasheet" ""
+			(at 179.07 67.31 0)
+			(hide yes)
+			(show_name no)
+			(do_not_autoplace no)
+			(effects
+				(font
+					(size 1.27 1.27)
+				)
+			)
+		)
+		(property "Description" "400W, 5V, Unidirectional, TVS"
+			(at 179.07 67.31 0)
+			(hide yes)
+			(show_name no)
+			(do_not_autoplace no)
+			(effects
+				(font
+					(size 1.27 1.27)
+				)
+				(justify bottom)
+			)
+		)
+		(property "MF" "Taiwan Semiconductor"
+			(at 179.07 67.31 0)
+			(hide yes)
+			(show_name no)
+			(do_not_autoplace no)
+			(effects
+				(font
+					(size 1.27 1.27)
+				)
+				(justify bottom)
+			)
+		)
+		(property "MAXIMUM_PACKAGE_HEIGHT" "2.5 mm"
+			(at 179.07 67.31 0)
+			(hide yes)
+			(show_name no)
+			(do_not_autoplace no)
+			(effects
+				(font
+					(size 1.27 1.27)
+				)
+				(justify bottom)
+			)
+		)
+		(property "Package" "SMA-2 Taiwan Semiconductor"
+			(at 179.07 67.31 0)
+			(hide yes)
+			(show_name no)
+			(do_not_autoplace no)
+			(effects
+				(font
+					(size 1.27 1.27)
+				)
+				(justify bottom)
+			)
+		)
+		(property "Price" "None"
+			(at 179.07 67.31 0)
+			(hide yes)
+			(show_name no)
+			(do_not_autoplace no)
+			(effects
+				(font
+					(size 1.27 1.27)
+				)
+				(justify bottom)
+			)
+		)
+		(property "Check_prices" "https://www.snapeda.com/parts/SMAJ5.0A/taiwan/view-part/?ref=eda"
+			(at 179.07 67.31 0)
+			(hide yes)
+			(show_name no)
+			(do_not_autoplace no)
+			(effects
+				(font
+					(size 1.27 1.27)
+				)
+				(justify bottom)
+			)
+		)
+		(property "STANDARD" "IPC-7351B"
+			(at 179.07 67.31 0)
+			(hide yes)
+			(show_name no)
+			(do_not_autoplace no)
+			(effects
+				(font
+					(size 1.27 1.27)
+				)
+				(justify bottom)
+			)
+		)
+		(property "PARTREV" "S2102"
+			(at 179.07 67.31 0)
+			(hide yes)
+			(show_name no)
+			(do_not_autoplace no)
+			(effects
+				(font
+					(size 1.27 1.27)
+				)
+				(justify bottom)
+			)
+		)
+		(property "SnapEDA_Link" "https://www.snapeda.com/parts/SMAJ5.0A/taiwan/view-part/?ref=snap"
+			(at 179.07 67.31 0)
+			(hide yes)
+			(show_name no)
+			(do_not_autoplace no)
+			(effects
+				(font
+					(size 1.27 1.27)
+				)
+				(justify bottom)
+			)
+		)
+		(property "MP" "SMAJ5.0A"
+			(at 179.07 67.31 0)
+			(hide yes)
+			(show_name no)
+			(do_not_autoplace no)
+			(effects
+				(font
+					(size 1.27 1.27)
+				)
+				(justify bottom)
+			)
+		)
+		(property "Availability" "In Stock"
+			(at 179.07 67.31 0)
+			(hide yes)
+			(show_name no)
+			(do_not_autoplace no)
+			(effects
+				(font
+					(size 1.27 1.27)
+				)
+				(justify bottom)
+			)
+		)
+		(property "MANUFACTURER" "Taiwan Semiconductor"
+			(at 179.07 67.31 0)
+			(hide yes)
+			(show_name no)
+			(do_not_autoplace no)
+			(effects
+				(font
+					(size 1.27 1.27)
+				)
+				(justify bottom)
+			)
+		)
+		(pin "A"
+		)
+		(pin "C"
+		)
+		(instances
+			(project "VENDETTAFC"
+				(path "/9ae0bade-d999-4f08-aa3a-8f8795024d1d/f4654729-a114-4964-8f4c-68feea8f16a2"
+					(reference "D5")
+					(unit 1)
+				)
+			)
+		)
+	)
+	(symbol
 		(lib_id "power:GND")
 		(at 241.3 195.58 0)
@@
 	)
 	(symbol
-		(lib_id "SMBJ30A:SMBJ30A")
-		(at 179.07 67.31 270)
-		(unit 1)
-		(body_style 1)
-		(exclude_from_sim no)
-		(in_bom yes)
-		(on_board yes)
-		(in_pos_files yes)
-		(dnp no)
-		(property "Reference" "D5"
-			(at 181.61 66.0399 90)
-			(show_name no)
-			(do_not_autoplace no)
-			(effects
-				(font
-					(size 1.27 1.27)
-				)
-				(justify left)
-			)
-		)
-		(property "Value" "SMBJ30A"
-			(at 181.356 68.326 90)
-			(show_name no)
-			(do_not_autoplace no)
-			(effects
-				(font
-					(size 1.27 1.27)
-				)
-				(justify left)
-			)
-		)
-		(property "Footprint" "SMBJ30A:DIOM4336X265N"
-			(at 179.07 67.31 0)
-			(hide yes)
-			(show_name no)
-			(do_not_autoplace no)
-			(effects
-				(font
-					(size 1.27 1.27)
-				)
-				(justify bottom)
-			)
-		)
-		(property "Datasheet" ""
-			(at 179.07 67.31 0)
-			(hide yes)
-			(show_name no)
-			(do_not_autoplace no)
-			(effects
-				(font
-					(size 1.27 1.27)
-				)
-			)
-		)
-		(property "Description" "600W, 30V, Unidirectional, TVS"
-			(at 179.07 67.31 0)
-			(hide yes)
-			(show_name no)
-			(do_not_autoplace no)
-			(effects
-				(font
-					(size 1.27 1.27)
-				)
-				(justify bottom)
-			)
-		)
-		(property "MF" "Taiwan Semiconductor"
-			(at 179.07 67.31 0)
-			(hide yes)
-			(show_name no)
-			(do_not_autoplace no)
-			(effects
-				(font
-					(size 1.27 1.27)
-				)
-				(justify bottom)
-			)
-		)
-		(property "MAXIMUM_PACKAGE_HEIGHT" "2.65 mm"
-			(at 179.07 67.31 0)
-			(hide yes)
-			(show_name no)
-			(do_not_autoplace no)
-			(effects
-				(font
-					(size 1.27 1.27)
-				)
-				(justify bottom)
-			)
-		)
-		(property "Package" "SMD-2 Taiwan Semiconductor"
-			(at 179.07 67.31 0)
-			(hide yes)
-			(show_name no)
-			(do_not_autoplace no)
-			(effects
-				(font
-					(size 1.27 1.27)
-				)
-				(justify bottom)
-			)
-		)
-		(property "Price" "None"
-			(at 179.07 67.31 0)
-			(hide yes)
-			(show_name no)
-			(do_not_autoplace no)
-			(effects
-				(font
-					(size 1.27 1.27)
-				)
-				(justify bottom)
-			)
-		)
-		(property "Check_prices" "https://www.snapeda.com/parts/SMBJ30A/taiwan/view-part/?ref=eda"
-			(at 179.07 67.31 0)
-			(hide yes)
-			(show_name no)
-			(do_not_autoplace no)
-			(effects
-				(font
-					(size 1.27 1.27)
-				)
-				(justify bottom)
-			)
-		)
-		(property "STANDARD" "IPC-7351B"
-			(at 179.07 67.31 0)
-			(hide yes)
-			(show_name no)
-			(do_not_autoplace no)
-			(effects
-				(font
-					(size 1.27 1.27)
-				)
-				(justify bottom)
-			)
-		)
-		(property "PARTREV" "F2102"
-			(at 179.07 67.31 0)
-			(hide yes)
-			(show_name no)
-			(do_not_autoplace no)
-			(effects
-				(font
-					(size 1.27 1.27)
-				)
-				(justify bottom)
-			)
-		)
-		(property "SnapEDA_Link" "https://www.snapeda.com/parts/SMBJ30A/taiwan/view-part/?ref=snap"
-			(at 179.07 67.31 0)
-			(hide yes)
-			(show_name no)
-			(do_not_autoplace no)
-			(effects
-				(font
-					(size 1.27 1.27)
-				)
-				(justify bottom)
-			)
-		)
-		(property "MP" "SMBJ30A"
-			(at 179.07 67.31 0)
-			(hide yes)
-			(show_name no)
-			(do_not_autoplace no)
-			(effects
-				(font
-					(size 1.27 1.27)
-				)
-				(justify bottom)
-			)
-		)
-		(property "Purchase-URL" "https://www.snapeda.com/api/url_track_click_mouser/?unipart_id=2759386&manufacturer=Taiwan Semiconductor&part_name=SMBJ30A&search_term=smbj30a"
-			(at 179.07 67.31 0)
-			(hide yes)
-			(show_name no)
-			(do_not_autoplace no)
-			(effects
-				(font
-					(size 1.27 1.27)
-				)
-				(justify bottom)
-			)
-		)
-		(property "Availability" "In Stock"
-			(at 179.07 67.31 0)
-			(hide yes)
-			(show_name no)
-			(do_not_autoplace no)
-			(effects
-				(font
-					(size 1.27 1.27)
-				)
-				(justify bottom)
-			)
-		)
-		(property "MANUFACTURER" "Taiwan Semiconductor"
-			(at 179.07 67.31 0)
-			(hide yes)
-			(show_name no)
-			(do_not_autoplace no)
-			(effects
-				(font
-					(size 1.27 1.27)
-				)
-				(justify bottom)
-			)
-		)
-		(pin "C"
-		)
-		(pin "A"
-		)
-		(instances
-			(project "VENDETTAFC"
-				(path "/9ae0bade-d999-4f08-aa3a-8f8795024d1d/f4654729-a114-4964-8f4c-68feea8f16a2"
-					(reference "D5")
-					(unit 1)
-				)
-			)
-		)
-	)
-	(symbol
 		(lib_id "Device:R")
 		(at 111.76 168.91 270)
@@
 			)
 		)
-		(property "Footprint" "Inductor_SMD:L_0402_1005Metric"
+		(property "Footprint" "Inductor_SMD:L_Changjiang_FTC404020S"
 			(at 137.16 163.83 0)
 			(hide yes)
@@
 			)
 		)
-		(property "Description" "Inductor"
+		(property "Description" "FAUKU GXTC0420-100-MT"
 			(at 137.16 163.83 0)
 			(hide yes)
@@
 			)
 		)
-		(property "Footprint" "Inductor_SMD:L_0402_1005Metric"
+		(property "Footprint" "Inductor_SMD:L_Changjiang_FTC404020S"
 			(at 311.15 163.83 0)
 			(hide yes)
@@
 			)
 		)
-		(property "Description" "Inductor"
+		(property "Description" "FAUKU GXTC0420-100-MT"
 			(at 311.15 163.83 0)
 			(hide yes)

Commit message: VFC Revision 2.0
Parts:
- added C45, C46, C47, C48: 0.1uF, Capacitor_SMD:C_0402_1005Metric, symbol Device:C
- added C49, C50: 100nF, Capacitor_SMD:C_0402_1005Metric, symbol Device:C
- C12, C13: footprint Capacitor_SMD:C_0402_1005Metric -> Capacitor_SMD:C_0603_1608Metric
- C17, C19, C20, C22: footprint Capacitor_SMD:C_0603_1608Metric -> Capacitor_SMD:C_0805_2012Metric
- C18, C21: value 100uF -> 10uF; footprint Capacitor_SMD:C_0603_1608Metric -> Capacitor_SMD:C_0805_2012Metric
Connections:
- net +3.3V: now also C50.1
- net +3.3VA: now also C49.1
- net +5VBAT: now also C48.1
- net +9V: now also C47.1
- net +VLIPO: now also C45.1, C46.1
- net GND: now also C45.2, C46.2, C47.2, C48.2, C49.2, C50.2
Other:
- moved on the sheet: C13, C17, C18

Commit message: Rev 2.0 fabrication documentation
Parts:
- C12, C13: Distributor Link (none) -> https://www.lcsc.com/product-detail/C19666.html?spm=wm.fly.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; LCSC (none) -> C19666; MANUFACTURER (none) -> Samsung Electro-Mechanics; MANUFACTURER PART NUMBER (none) -> CL10A475KO8NNNC
- C14, C15, C32, C49, C50: Distributor Link (none) -> https://www.lcsc.com/product-detail/C100072.html?spm=wm.fly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; LCSC (none) -> C100072; MANUFACTURER (none) -> Samsung Electro-Mechanics; MANUFACTURER PART NUMBER (none) -> CL05A104KA5NNNC
- C17, C19: Distributor Link (none) -> https://www.lcsc.com/product-detail/C22367832.html?spm=wm.f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; LCSC (none) -> C22367832; MANUFACTURER (none) -> Chinocera; MANUFACTURER PART NUMBER (none) -> HGC0805R5226M350NSLJ
- C18, C21: Distributor Link (none) -> https://www.lcsc.com/product-detail/C2932476.html?spm=wm.fl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; LCSC (none) -> C2932476; MANUFACTURER (none) -> Samsung Electro-Mechanics; MANUFACTURER PART NUMBER (none) -> CL21A106KBYQNNE
- C20, C22: Distributor Link (none) -> https://www.lcsc.com/product-detail/C5596752.html?spm=wm.fl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; LCSC (none) -> C5596752; MANUFACTURER (none) -> Samsung Electro-Mechanics; MANUFACTURER PART NUMBER (none) -> CL21A476MPYNNWE
- C24, C25, C39: Distributor Link (none) -> https://www.lcsc.com/product-detail/C29266.html?spm=wm.fly.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; LCSC (none) -> C29266; MANUFACTURER (none) -> Samsung Electro-Mechanics; MANUFACTURER PART NUMBER (none) -> CL05A105KO5NNNC
- C41, C42, C45, C46, C47, C48: value 0.1uF -> 100nF; Distributor Link (none) -> https://www.lcsc.com/product-detail/C100072.html?spm=wm.fly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; LCSC (none) -> C100072; MANUFACTURER (none) -> Samsung Electro-Mechanics; MANUFACTURER PART NUMBER (none) -> CL05A104KA5NNNC
- D5: Distributor Link (none) -> https://www.lcsc.com/product-detail/C83329.html?s_z=s_p_x_S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; LCSC (none) -> C83329; MANUFACTURER Taiwan Semiconductor -> Littelfuse; MANUFACTURER PART NUMBER (none) -> SMAJ5.0A
- D7: Distributor Link (none) -> https://www.lcsc.com/product-detail/C2286.html?s_z=s_p_KT-0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; LCSC (none) -> C2286; MANUFACTURER PART NUMBER (none) -> KT-0603R
- D8: Distributor Link (none) -> https://www.lcsc.com/product-detail/C14308.html?s_z=s_q_x_B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; LCSC (none) -> C14308; MANUFACTURER (none) -> onsemi; MANUFACTURER PART NUMBER (none) -> BAT54CLT1G
- F2: Distributor Link (none) -> https://www.lcsc.com/product-detail/C2649903.html?spm=wm.fl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; LCSC (none) -> C2649903; MANUFACTURER (none) -> Littelfuse; MANUFACTURER PART NUMBER (none) -> MICROSMD010F-2
- FL2: footprint BLM18PG221SN1D:BEADC1608X95N -> Inductor_SMD:L_0402_1005Metric; Distributor Link (none) -> https://www.lcsc.com/product-detail/C85818.html?s_z=n_q_t_f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; LCSC (none) -> C85818; MANUFACTURER (none) -> muRata; MANUFACTURER PART NUMBER (none) -> BLM15BB221SN1D
- J2: Distributor Link (none) -> https://www.lcsc.com/product-detail/C54829818.html?s_z=n_q_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; LCSC (none) -> C54829818; MANUFACTURER Global Connector Technology -> YUWENFA; MANUFACTURER PART NUMBER (none) -> PTCFW-H22S-001
- L1, L2: Distributor Link (none) -> https://www.lcsc.com/product-detail/C53198553.html?s_z=s_p_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; LCSC (none) -> C53198553; MANUFACTURER (none) -> FAUKU; MANUFACTURER PART NUMBER (none) -> GXTC0420-100-MT
- R1, R5: Distributor Link (none) -> https://www.lcsc.com/product-detail/C105872.html?spm=wm.fly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; LCSC (none) -> C105872; MANUFACTURER (none) -> YAGEO; MANUFACTURER PART NUMBER (none) -> RC0402FR-075K1L
- R10, R13: Distributor Link (none) -> https://www.lcsc.com/product-detail/C138031.html?spm=wm.fly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; LCSC (none) -> C138031; MANUFACTURER (none) -> YAGEO; MANUFACTURER PART NUMBER (none) -> RC0402FR-0720RL
- R11: Distributor Link (none) -> https://www.lcsc.com/product-detail/C25762.html?spm=wm.fly.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; LCSC (none) -> C25762; MANUFACTURER (none) -> UNI-ROYAL; MANUFACTURER PART NUMBER (none) -> 0402WGF1802TCE
- R14, R7: Distributor Link (none) -> https://www.lcsc.com/product-detail/C107229.html?spm=wm.fly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; LCSC (none) -> C107229; MANUFACTURER (none) -> YAGEO; MANUFACTURER PART NUMBER (none) -> RC0402FR-0751KL
- R15: Distributor Link (none) -> https://www.lcsc.com/product-detail/C25918.html?spm=wm.fly.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; LCSC (none) -> C25918; MANUFACTURER (none) -> UNI-ROYAL; MANUFACTURER PART NUMBER (none) -> 0402WGF7501TCE
- R16, R8: Distributor Link (none) -> https://www.lcsc.com/product-detail/C844310.html?spm=wm.fly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; LCSC (none) -> C844310; MANUFACTURER (none) -> VISHAY; MANUFACTURER PART NUMBER (none) -> CRCW040241K2FKED
- R17: Distributor Link (none) -> https://www.lcsc.com/product-detail/C60488.html?spm=wm.fly.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; LCSC (none) -> C60488; MANUFACTURER (none) -> YAGEO; MANUFACTURER PART NUMBER (none) -> RC0402FR-072KL
- R2, R3: Distributor Link (none) -> https://www.lcsc.com/product-detail/C185392.html?spm=wm.fly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; LCSC (none) -> C185392; MANUFACTURER (none) -> YAGEO; MANUFACTURER PART NUMBER (none) -> RC0402FR-0780R6L
- R31: Distributor Link (none) -> https://www.lcsc.com/product-detail/C112291.html?spm=wm.fly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; LCSC (none) -> C112291; MANUFACTURER (none) -> YAGEO; MANUFACTURER PART NUMBER (none) -> RC0402FR-07220RL
- R32: value 5.1K -> 5k1; Distributor Link (none) -> https://www.lcsc.com/product-detail/C105872.html?spm=wm.fly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; LCSC (none) -> C105872; MANUFACTURER (none) -> YAGEO; MANUFACTURER PART NUMBER (none) -> RC0402FR-075K1L
- R33: Distributor Link (none) -> https://www.lcsc.com/product-detail/C60489.html?spm=wm.fly.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; LCSC (none) -> C60489; MANUFACTURER (none) -> YAGEO; MANUFACTURER PART NUMBER (none) -> RC0402JR-0710KL
- R36, R37: Distributor Link (none) -> https://www.lcsc.com/product-detail/C93949.html?spm=wm.fly.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; LCSC (none) -> C93949; MANUFACTURER (none) -> YAGEO; MANUFACTURER PART NUMBER (none) -> RC0402JR-071ML
- R9: Distributor Link (none) -> https://www.lcsc.com/product-detail/C131467.html?spm=wm.fly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; LCSC (none) -> C131467; MANUFACTURER (none) -> YAGEO; MANUFACTURER PART NUMBER (none) -> RC0402FR-073K9L
- U10: Distributor Link (none) -> https://www.lcsc.com/product-detail/C7519.html?s_z=s_p_USBL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; LCSC (none) -> C7519; MANUFACTURER (none) -> ST; MANUFACTURER PART NUMBER (none) -> USBLC6-2SC6
- U11: value AP7361C-FGE-7 -> AP7361C-33FGE-7; Distributor Link (none) -> https://www.lcsc.com/product-detail/C151007.html?s_z=s_p_AP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; LCSC (none) -> C151007; MANUFACTURER PART NUMBER (none) -> AP7361C-33FGE-7
- U3: Distributor Link (none) -> https://www.lcsc.com/product-detail/C892227.html?s_z=s_p_NC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; LCSC (none) -> C892227; MANUFACTURER PART NUMBER (none) -> NCP167BMX330TBG
- U4, U9: value (none) -> MP9943GQ-Z; Distributor Link (none) -> https://www.mouser.in/ProductDetail/Monolithic-Power-System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; LCSC (none) -> Mouser No: 946-MP9943GQ-Z; MANUFACTURER (none) -> Monolithic Power Systems (MPS); MANUFACTURER PART NUMBER (none) -> MP9943GQ-Z
