File: VFC/sensor.kicad_sch (KiCad schematic)
At the start: 44 parts, among them Q2 AO3400A, U2 BMP388, U5 ESP32-C3, U6 ICM-42688-P, U7 W25N04KVZEIR, Y2 C3E-40.000-10-1015-X-R

Commit message: LICENSE
Parts:
- removed R19, R30: 10K, Resistor_SMD:R_0402_1005Metric, symbol Device:R
- added R6: 10K, Resistor_SMD:R_0402_1005Metric, symbol Device:R
Connections:
- net ESP_CS is gone; now on an unnamed net: U5.20 (GPIO13/SPIWP)
- net ESP_MISO is gone; now on an unnamed net: U5.21 (GPIO14/SPICS0)
- net +3.3V: now also R6.1; no longer U5.7 (CHIP_EN)
- net ESP_BOOT: now reaches U5.15 (GPIO9)
- net at TP1.1: no longer U5.27 (GPIO20/U0RXD)
- net at TP2.1: no longer U5.28 (GPIO21/U0TXD)
- net ESP_MOSI: no longer names the net of U5.23 (GPIO16/SPID)
- net ESP_SCK: no longer names the net of U5.22 (GPIO15/SPICLK)
- new net ESP_EN: R6.2, U5.7 (CHIP_EN)
- new net ESP_RX: U5.28 (GPIO21/U0TXD)
- new net ESP_TX: U5.27 (GPIO20/U0RXD)
- no-connect marks 18 -> 20

Commit message: Routing improvements
Parts:
- removed C30, C31: 1pF, Capacitor_SMD:C_0402_1005Metric, symbol Device:C
- removed U8: (no value), crossair-ca-c03-antenna-1.snapshot.1:CA-C03, symbol CA-C03:CA-C03
- added AT1: 2450AT43B100E, 2450AT43B100E:ANTENNA_2450AT43B100E, symbol 2450AT43B100E:2450AT43B100E
- L3: value 2nH -> 1.8nH
Connections:
- net ANT: now also AT1.1
Other:
- moved on the sheet: Q2, R34, R35

Commit message: Routing improvements
Connections:
- net FLS_MISO renamed FLS/OSD_MOSI
- net FLS_MOSI renamed FLS/OSD_MISO
- net FLS_SCK renamed FLS/OSD_SCK
Changed lines of the file:
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@@
 		)
 	)
-	(global_label "FLS_MISO"
+	(global_label "FLS{slash}OSD_MISO"
+		(shape input)
+		(at 111.76 147.32 0)
+		(fields_autoplaced yes)
+		(effects
+			(font
+				(size 1.27 1.27)
+			)
+			(justify left)
+		)
+		(property "Intersheetrefs" "${INTERSHEET_REFS}"
+			(at 128.7757 147.32 0)
+			(hide yes)
+			(show_name no)
+			(do_not_autoplace no)
+			(effects
+				(font
+					(size 1.27 1.27)
+				)
+				(justify left)
+			)
+		)
+	)
+	(global_label "IMU_MOSI"
+		(shape input)
+		(at 63.5 77.47 180)
+		(fields_autoplaced yes)
+		(effects
+			(font
+				(size 1.27 1.27)
+			)
+			(justify right)
+		)
+		(property "Intersheetrefs" "${INTERSHEET_REFS}"
+			(at 51.5643 77.47 0)
+			(hide yes)
+			(show_name no)
+			(do_not_autoplace no)
+			(effects
+				(font
+					(size 1.27 1.27)
+				)
+				(justify right)
+			)
+		)
+	)
+	(global_label "BAR_SCL"
+		(shape input)
+		(at 77.47 223.52 180)
+		(fields_autoplaced yes)
+		(effects
+			(font
+				(size 1.27 1.27)
+			)
+			(justify right)
+		)
+		(property "Intersheetrefs" "${INTERSHEET_REFS}"
+			(at 66.381 223.52 0)
+			(hide yes)
+			(show_name no)
+			(do_not_autoplace no)
+			(effects
+				(font
+					(size 1.27 1.27)
+				)
+				(justify right)
+			)
+		)
+	)
+	(global_label "FLS_CS"
+		(shape input)
+		(at 53.34 147.32 180)
+		(fields_autoplaced yes)
+		(effects
+			(font
+				(size 1.27 1.27)
+			)
+			(justify right)
+		)
+		(property "Intersheetrefs" "${INTERSHEET_REFS}"
+			(at 43.5815 147.32 0)
+			(hide yes)
+			(show_name no)
+			(do_not_autoplace no)
+			(effects
+				(font
+					(size 1.27 1.27)
+				)
+				(justify right)
+			)
+		)
+	)
+	(global_label "FLS{slash}OSD_MOSI"
 		(shape input)
 		(at 111.76 149.86 0)
@@
 		)
 		(property "Intersheetrefs" "${INTERSHEET_REFS}"
-			(at 123.6352 149.86 0)
-			(hide yes)
-			(show_name no)
-			(do_not_autoplace no)
-			(effects
-				(font
-					(size 1.27 1.27)
-				)
-				(justify left)
-			)
-		)
-	)
-	(global_label "FLS_MOSI"
-		(shape input)
-		(at 111.76 147.32 0)
-		(fields_autoplaced yes)
-		(effects
-			(font
-				(size 1.27 1.27)
-			)
-			(justify left)
-		)
-		(property "Intersheetrefs" "${INTERSHEET_REFS}"
-			(at 123.6352 147.32 0)
-			(hide yes)
-			(show_name no)
-			(do_not_autoplace no)
-			(effects
-				(font
-					(size 1.27 1.27)
-				)
-				(justify left)
-			)
-		)
-	)
-	(global_label "IMU_MOSI"
-		(shape input)
-		(at 63.5 77.47 180)
-		(fields_autoplaced yes)
-		(effects
-			(font
-				(size 1.27 1.27)
-			)
-			(justify right)
-		)
-		(property "Intersheetrefs" "${INTERSHEET_REFS}"
-			(at 51.5643 77.47 0)
-			(hide yes)
-			(show_name no)
-			(do_not_autoplace no)
-			(effects
-				(font
-					(size 1.27 1.27)
-				)
-				(justify right)
-			)
-		)
-	)
-	(global_label "BAR_SCL"
-		(shape input)
-		(at 77.47 223.52 180)
-		(fields_autoplaced yes)
-		(effects
-			(font
-				(size 1.27 1.27)
-			)
-			(justify right)
-		)
-		(property "Intersheetrefs" "${INTERSHEET_REFS}"
-			(at 66.381 223.52 0)
-			(hide yes)
-			(show_name no)
-			(do_not_autoplace no)
-			(effects
-				(font
-					(size 1.27 1.27)
-				)
-				(justify right)
-			)
-		)
-	)
-	(global_label "FLS_CS"
-		(shape input)
-		(at 53.34 147.32 180)
-		(fields_autoplaced yes)
-		(effects
-			(font
-				(size 1.27 1.27)
-			)
-			(justify right)
-		)
-		(property "Intersheetrefs" "${INTERSHEET_REFS}"
-			(at 43.5815 147.32 0)
+			(at 128.7757 149.86 0)
+			(hide yes)
+			(show_name no)
+			(do_not_autoplace no)
+			(effects
+				(font
+					(size 1.27 1.27)
+				)
+				(justify left)
+			)
+		)
+	)
+	(global_label "FLS{slash}OSD_SCK"
+		(shape input)
+		(at 53.34 149.86 180)
+		(fields_autoplaced yes)
+		(effects
+			(font
+				(size 1.27 1.27)
+			)
+			(justify right)
+		)
+		(property "Intersheetrefs" "${INTERSHEET_REFS}"
+			(at 37.171 149.86 0)
 			(hide yes)
 			(show_name no)
@@
 			)
 		)
-	)
-	(global_label "FLS_SCK"
-		(shape input)
-		(at 53.34 149.86 180)
-		(fields_autoplaced yes)
-		(effects
-			(font
-				(size 1.27 1.27)
-			)
-			(justify right)
-		)
-		(property "Intersheetrefs" "${INTERSHEET_REFS}"
-			(at 42.3115 149.86 0)
-			(hide yes)
-			(show_name no)
-			(do_not_autoplace no)
-			(effects
-				(font
-					(size 1.27 1.27)
-				)
-				(justify right)
-			)
-		)

Commit message: Rev 2.0 fabrication documentation
Parts:
- AT1: Distributor Link (none) -> https://www.lcsc.com/product-detail/C2917721.html?s_z=s_p_2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; LCSC (none) -> C2917721; MANUFACTURER Johanson Technology Inc. -> Johanson Dielectrics; MANUFACTURER PART NUMBER (none) -> 2450AT43B100E
- C10, C33: Distributor Link (none) -> https://www.lcsc.com/product-detail/C15195.html?spm=wm.fly.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; LCSC (none) -> C15195; MANUFACTURER (none) -> Samsung Electro-Mechanics; MANUFACTURER PART NUMBER (none) -> CL05B103KB5NNNC
- C11, C28, C38: Distributor Link (none) -> https://www.lcsc.com/product-detail/C100072.html?spm=wm.fly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; LCSC (none) -> C100072; MANUFACTURER (none) -> Samsung Electro-Mechanics; MANUFACTURER PART NUMBER (none) -> CL05A104KA5NNNC
- C29, C35, C36, C4: value 0.1uF -> 100nF; Distributor Link (none) -> https://www.lcsc.com/product-detail/C100072.html?spm=wm.fly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; LCSC (none) -> C100072; MANUFACTURER (none) -> Samsung Electro-Mechanics; MANUFACTURER PART NUMBER (none) -> CL05A104KA5NNNC
- C34: Distributor Link (none) -> https://www.lcsc.com/product-detail/C29266.html?spm=wm.fly.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; LCSC (none) -> C29266; MANUFACTURER (none) -> Samsung Electro-Mechanics; MANUFACTURER PART NUMBER (none) -> CL05A105KO5NNNC
- C37: footprint Capacitor_SMD:C_0603_1608Metric -> Capacitor_SMD:C_0805_2012Metric; Distributor Link (none) -> https://www.lcsc.com/product-detail/C2932476.html?spm=wm.fl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; LCSC (none) -> C2932476; MANUFACTURER (none) -> Samsung Electro-Mechanics; MANUFACTURER PART NUMBER (none) -> CL21A106KBYQNNE
- C9: Distributor Link (none) -> https://www.lcsc.com/product-detail/C107369.html?spm=wm.fly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; LCSC (none) -> C107369; MANUFACTURER (none) -> Samsung Electro-Mechanics; MANUFACTURER PART NUMBER (none) -> CL05A225KP5NSNC
- D1: Distributor Link (none) -> https://www.lcsc.com/product-detail/C2293.html?s_z=n_q_KT-0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; LCSC (none) -> C2293; MANUFACTURER (none) -> Hubei KENTO Elec; MANUFACTURER PART NUMBER (none) -> KT-0805B
- D2: Distributor Link (none) -> https://www.lcsc.com/product-detail/C2296.html?s_z=n_q_KT-0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; LCSC (none) -> C2296; MANUFACTURER (none) -> Hubei KENTO Elec; MANUFACTURER PART NUMBER (none) -> KT-0805Y
- D3: Distributor Link (none) -> https://www.lcsc.com/product-detail/C2297.html?s_z=n_q_KT-0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; LCSC (none) -> C2297; MANUFACTURER (none) -> Hubei KENTO Elec; MANUFACTURER PART NUMBER (none) -> KT-0805G
- D4: Distributor Link (none) -> https://www.lcsc.com/product-detail/C2295.html?s_z=n_q_KT-0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; LCSC (none) -> C2295; MANUFACTURER (none) -> Hubei KENTO Elec; MANUFACTURER PART NUMBER (none) -> KT-0805R
- L3: Distributor Link (none) -> https://www.lcsc.com/product-detail/C77107.html?s_z=s_p_LQG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; LCSC (none) -> C77107; MANUFACTURER (none) -> muRata; MANUFACTURER PART NUMBER (none) -> LQG15HS1N8S02D
- Q2: Distributor Link (none) -> https://www.lcsc.com/product-detail/C20917.html?s_z=s_p_AO3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; LCSC (none) -> C20917; MANUFACTURER (none) -> AOS; MANUFACTURER PART NUMBER (none) -> AO3400A
- R12, R20, R35, R4, R6: Distributor Link (none) -> https://www.lcsc.com/product-detail/C60489.html?spm=wm.fly.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; LCSC (none) -> C60489; MANUFACTURER (none) -> YAGEO; MANUFACTURER PART NUMBER (none) -> RC0402JR-0710KL
- R18: Distributor Link (none) -> https://www.lcsc.com/product-detail/C137973.html?spm=wm.fly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; LCSC (none) -> C137973; MANUFACTURER (none) -> YAGEO; MANUFACTURER PART NUMBER (none) -> RC0402FR-0747RL
- R21: Distributor Link (none) -> https://www.lcsc.com/product-detail/C112291.html?spm=wm.fly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; LCSC (none) -> C112291; MANUFACTURER (none) -> YAGEO; MANUFACTURER PART NUMBER (none) -> RC0402FR-07220RL
- R22, R34: Distributor Link (none) -> https://www.lcsc.com/product-detail/C106235.html?spm=wm.fly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; LCSC (none) -> C106235; MANUFACTURER (none) -> YAGEO; MANUFACTURER PART NUMBER (none) -> RC0402FR-071KL
- R23: Distributor Link (none) -> https://www.lcsc.com/product-detail/C137841.html?spm=wm.fly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; LCSC (none) -> C137841; MANUFACTURER (none) -> YAGEO; MANUFACTURER PART NUMBER (none) -> RC0402JR-0775RL
- R25, R26: Distributor Link (none) -> https://www.lcsc.com/product-detail/C163447.html?spm=wm.fly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; LCSC (none) -> C163447; MANUFACTURER (none) -> YAGEO; MANUFACTURER PART NUMBER (none) -> RC0402JR-072K2L
- R27, R28, R29: Distributor Link (none) -> https://www.lcsc.com/product-detail/C105871.html?spm=wm.fly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; LCSC (none) -> C105871; MANUFACTURER (none) -> YAGEO; MANUFACTURER PART NUMBER (none) -> RC0402FR-074K7L
- TP1, TP2: Distributor Link (none) -> -; LCSC (none) -> -; MANUFACTURER (none) -> -; MANUFACTURER PART NUMBER (none) -> -
- U2: Distributor Link (none) -> https://www.lcsc.com/product-detail/C779278.html?s_z=s_p_x_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; LCSC (none) -> C779278; MANUFACTURER PART NUMBER (none) -> BMP388
- U5: Distributor Link (none) -> https://www.lcsc.com/product-detail/C2838500.html?s_z=s_p_x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; LCSC (none) -> C2838500; MANUFACTURER PART NUMBER (none) -> ESP32-C3
- U6: Distributor Link (none) -> https://www.lcsc.com/product-detail/C1850418.html?s_z=s_p_t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; LCSC (none) -> C1850418, Mouser No: 410-ICM-42688-P; MANUFACTURER PART NUMBER (none) -> ICM-42688-P
- U7: value W25N04KVZEIR -> W25Q256JVEIQ; Distributor Link (none) -> https://www.lcsc.com/product-detail/C97522.html?s_z=n_q_W25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; LCSC (none) -> C97522; MANUFACTURER PART NUMBER (none) -> W25Q256JVEIQ
- Y2: Distributor Link (none) -> https://www.lcsc.com/product-detail/C5444549.html?s_z=n_q_%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; LCSC (none) -> C5444549; MANUFACTURER Aker -> YXC Crystal Oscillators; MANUFACTURER PART NUMBER (none) -> XL2EL89CPI-111YLC-40M
